Commit message: Simplify collision mesh

File: op3_description/urdf/robotis_op3.structure.head.xacro (robot description, xacro)
@@ -22,5 +22,5 @@
       </visual>
       <collision>
-        <xacro:insert_mesh_head_pan_link/>
+        <xacro:insert_box_head_pan_link/>
       </collision>
       <inertial>
@@ -44,5 +44,5 @@
       </visual>
       <collision>
-        <xacro:insert_mesh_head_tilt_link/>
+        <xacro:insert_box_head_tilt_link/>
       </collision>
       <inertial>

File: op3_description/urdf/robotis_op3.structure.larm.xacro (robot description, xacro)
@@ -22,5 +22,5 @@
       </visual>
       <collision>
-        <xacro:insert_mesh_l_sho_pitch_link/>
+        <xacro:insert_box_l_sho_pitch_link/>
       </collision>
       <inertial>
@@ -44,5 +44,5 @@
       </visual>
       <collision>
-        <xacro:insert_mesh_l_sho_roll_link/>
+        <xacro:insert_box_l_sho_roll_link/>
       </collision>
       <inertial>
@@ -66,5 +66,5 @@
       </visual>
       <collision>
-        <xacro:insert_mesh_l_el_link/>
+        <xacro:insert_box_l_el_link/>
       </collision>
       <inertial>

File: op3_description/urdf/robotis_op3.structure.lleg.xacro (robot description, xacro)
@@ -22,5 +22,5 @@
       </visual>
       <collision>
-        <xacro:insert_mesh_l_hip_yaw_link/>
+        <xacro:insert_box_l_hip_yaw_link/>
       </collision>
       <inertial>
@@ -44,5 +44,5 @@
       </visual>
       <collision>
-        <xacro:insert_mesh_l_hip_roll_link/>
+        <xacro:insert_box_l_hip_roll_link/>
       </collision>
       <inertial>
@@ -66,5 +66,5 @@
       </visual>
       <collision>
-        <xacro:insert_mesh_l_hip_pitch_link/>
+        <xacro:insert_box_l_hip_pitch_link/>
       </collision>
       <inertial>
@@ -88,5 +88,5 @@
       </visual>
       <collision>
-        <xacro:insert_mesh_l_knee_link/>
+        <xacro:insert_box_l_knee_link/>
       </collision>
       <inertial>
@@ -110,5 +110,5 @@
       </visual>
       <collision>
-        <xacro:insert_mesh_l_ank_pitch_link/>
+        <xacro:insert_box_l_ank_pitch_link/>
       </collision>
       <inertial>
@@ -132,5 +132,5 @@
       </visual>
       <collision>
-        <xacro:insert_mesh_l_ank_roll_link/>
+        <xacro:insert_box_l_ank_roll_link/>
       </collision>
       <inertial>

File: op3_description/urdf/robotis_op3.structure.rarm.xacro (robot description, xacro)
@@ -22,5 +22,5 @@
       </visual>
       <collision>
-        <xacro:insert_mesh_r_sho_pitch_link/>
+        <xacro:insert_box_r_sho_pitch_link/>
       </collision>
       <inertial>
@@ -44,5 +44,5 @@
       </visual>
       <collision>
-        <xacro:insert_mesh_r_sho_roll_link/>
+        <xacro:insert_box_r_sho_roll_link/>
       </collision>
       <inertial>
@@ -66,5 +66,5 @@
       </visual>
       <collision>
-        <xacro:insert_mesh_r_el_link/>
+        <xacro:insert_box_r_el_link/>
       </collision>
       <inertial>

File: op3_description/urdf/robotis_op3.structure.rleg.xacro (robot description, xacro)
@@ -22,5 +22,5 @@
       </visual>
       <collision>
-        <xacro:insert_mesh_r_hip_yaw_link/>
+        <xacro:insert_box_r_hip_yaw_link/>
       </collision>
       <inertial>
@@ -44,5 +44,5 @@
       </visual>
       <collision>
-        <xacro:insert_mesh_r_hip_roll_link/>
+        <xacro:insert_box_r_hip_roll_link/>
       </collision>
       <inertial>
@@ -66,5 +66,5 @@
       </visual>
       <collision>
-        <xacro:insert_mesh_r_hip_pitch_link/>
+        <xacro:insert_box_r_hip_pitch_link/>
       </collision>
       <inertial>
@@ -88,5 +88,5 @@
       </visual>
       <collision>
-        <xacro:insert_mesh_r_knee_link/>
+        <xacro:insert_box_r_knee_link/>
       </collision>
       <inertial>
@@ -110,5 +110,5 @@
       </visual>
       <collision>
-        <xacro:insert_mesh_r_ank_pitch_link/>
+        <xacro:insert_box_r_ank_pitch_link/>
       </collision>
       <inertial>
@@ -132,5 +132,5 @@
       </visual>
       <collision>
-        <xacro:insert_mesh_r_ank_roll_link/>
+        <xacro:insert_box_r_ank_roll_link/>
       </collision>
       <inertial>

File: op3_description/urdf/robotis_op3.urdf.xacro (robot description, xacro)
@@ -39,5 +39,5 @@
     </visual>
     <collision>
-      <xacro:insert_mesh_body_link/>
+      <xacro:insert_box_body_link/>
     </collision>
     <inertial>

File: op3_description/urdf/robotis_op3.visuals.xacro (robot description, xacro)
@@ -14,4 +14,10 @@
     </material>
   </xacro:macro>
+  <xacro:macro name="insert_box_body_link">
+    <origin xyz="-0.0168 0.0000 0.0683" rpy="0.0000 -0.0000 -0.0000"/>
+    <geometry>
+      <box size="0.1745 0.1288 0.1453"/>
+    </geometry>
+  </xacro:macro>
   <!-- right hip yaw link -->
   <xacro:macro name="insert_mesh_r_hip_yaw_link">
@@ -24,4 +30,10 @@
     </material>
   </xacro:macro>
+  <xacro:macro name="insert_box_r_hip_yaw_link">
+    <origin xyz="-0.0015 0.0000 -0.0155" rpy="0.0000 -0.0000 -0.0000"/>
+    <geometry>
+      <box size="0.0450 0.0250 0.0310"/>
+    </geometry>
+  </xacro:macro>
   <!-- right hip roll link -->
   <xacro:macro name="insert_mesh_r_hip_roll_link">
@@ -34,4 +46,10 @@
     </material>
   </xacro:macro>
+  <xacro:macro name="insert_box_r_hip_roll_link">
+    <origin xyz="0.0039 -0.0022 -0.0120" rpy="0.0000 -0.0000 -0.0000"/>
+    <geometry>
+      <box size="0.0798 0.0424 0.0465"/>
+    </geometry>
+  </xacro:macro>
   <!-- right hip pitch link -->
   <xacro:macro name="insert_mesh_r_hip_pitch_link">
@@ -44,4 +62,10 @@
     </material>
   </xacro:macro>
+  <xacro:macro name="insert_box_r_hip_pitch_link">
+    <origin xyz="0.0004 0.0188 -0.0595" rpy="0.0000 -0.0000 -0.0000"/>
+    <geometry>
+      <box size="0.0309 0.0464 0.1239"/>
+    </geometry>
+  </xacro:macro>
   <!-- right knee link -->
   <xacro:macro name="insert_mesh_r_knee_link">
@@ -54,4 +78,10 @@
     </material>
   </xacro:macro>
+  <xacro:macro name="insert_box_r_knee_link">
+    <origin xyz="0.0000 0.0200 -0.0550" rpy="0.0000 -0.0000 -0.0000"/>
+    <geometry>
+      <box size="0.0300 0.0440 0.1150"/>
+    </geometry>
+  </xacro:macro>
   <!-- right ankle pitch link -->
   <xacro:macro name="insert_mesh_r_ank_pitch_link">
@@ -64,4 +94,10 @@
     </material>
   </xacro:macro>
+  <xacro:macro name="insert_box_r_ank_pitch_link">
+    <origin xyz="-0.0202 0.0168 0.0120" rpy="0.0000 -0.0000 -0.0000"/>
+    <geometry>
+      <box size="0.0798 0.0424 0.0465"/>
+    </geometry>
+  </xacro:macro>
   <!-- right ankle roll link -->
   <xacro:macro name="insert_mesh_r_ank_roll_link">
@@ -74,4 +110,10 @@
     </material>
   </xacro:macro>
+  <xacro:macro name="insert_box_r_ank_roll_link">
+    <origin xyz="0.0240 -0.0125 -0.0140" rpy="0.0000 -0.0000 -0.0000"/>
+    <geometry>
+      <box size="0.1270 0.0800 0.0330"/>
+    </geometry>
+  </xacro:macro>
   <!-- left hip yaw link -->
   <xacro:macro name="insert_mesh_l_hip_yaw_link">
@@ -84,4 +126,10 @@
     </material>
   </xacro:macro>
+  <xacro:macro name="insert_box_l_hip_yaw_link">
+    <origin xyz="-0.0015 0.0000 -0.0155" rpy="0.0000 -0.0000 -0.0000"/>
+    <geometry>
+      <box size="0.0450 0.0250 0.0310"/>
+    </geometry>
+  </xacro:macro>
   <!-- left hip roll link -->
   <xacro:macro name="insert_mesh_l_hip_roll_link">
@@ -94,4 +142,10 @@
     </material>
   </xacro:macro>
+  <xacro:macro name="insert_box_l_hip_roll_link">
+    <origin xyz="0.0039 0.0022 -0.0120" rpy="0.0000 -0.0000 -0.0000"/>
+    <geometry>
+      <box size="0.0798 0.0424 0.0465"/>
+    </geometry>
+  </xacro:macro>
   <!-- left hip pitch link -->
   <xacro:macro name="insert_mesh_l_hip_pitch_link">
@@ -104,4 +158,10 @@
     </material>
   </xacro:macro>
+  <xacro:macro name="insert_box_l_hip_pitch_link">
+    <origin xyz="0.0004 -0.0188 -0.0595" rpy="0.0000 -0.0000 -0.0000"/>
+    <geometry>
+      <box size="0.0309 0.0464 0.1239"/>
+    </geometry>
+  </xacro:macro>
   <!-- left knee link -->
   <xacro:macro name="insert_mesh_l_knee_link">
@@ -114,4 +174,10 @@
     </material>
   </xacro:macro>
+  <xacro:macro name="insert_box_l_knee_link">
+    <origin xyz="-0.0000 -0.0200 -0.0550" rpy="0.0000 -0.0000 -0.0000"/>
+    <geometry>
+      <box size="0.0300 0.0440 0.1150"/>
+    </geometry>
+  </xacro:macro>
   <!-- left ankle pitch link -->
   <xacro:macro name="insert_mesh_l_ank_pitch_link">
@@ -124,4 +190,10 @@
     </material>
   </xacro:macro>
+  <xacro:macro name="insert_box_l_ank_pitch_link">
+    <origin xyz="-0.0206 -0.0168 0.0120" rpy="0.0000 -0.0000 -0.0000"/>
+    <geometry>
+      <box size="0.0790 0.0424 0.0465"/>
+    </geometry>
+  </xacro:macro>
   <!-- left ankle roll link -->
   <xacro:macro name="insert_mesh_l_ank_roll_link">
@@ -134,4 +206,10 @@
     </material>
   </xacro:macro>
+  <xacro:macro name="insert_box_l_ank_roll_link">
+    <origin xyz="0.0240 0.0125 -0.0140" rpy="0.0000 -0.0000 -0.0000"/>
+    <geometry>
+      <box size="0.1270 0.0800 0.0330"/>
+    </geometry>
+  </xacro:macro>
   <!-- right shoulder pitch joint -->
   <xacro:macro name="insert_mesh_r_sho_pitch_link">
@@ -144,4 +222,10 @@
     </material>
   </xacro:macro>
+  <xacro:macro name="insert_box_r_sho_pitch_link">
+    <origin xyz="-0.0000 -0.0155 -0.0038" rpy="0.0000 -0.0000 -0.0000"/>
+    <geometry>
+      <box size="0.0420 0.0310 0.0325"/>
+    </geometry>
+  </xacro:macro>
   <!-- right shoulder pitch joint -->
   <xacro:macro name="insert_mesh_r_sho_roll_link">
@@ -154,4 +238,10 @@
     </material>
   </xacro:macro>
+  <xacro:macro name="insert_box_r_sho_roll_link">
+    <origin xyz="-0.0168 -0.0452 0.0007" rpy="0.0000 -0.0000 -0.0000"/>
+    <geometry>
+      <box size="0.0424 0.1129 0.0301"/>
+    </geometry>
+  </xacro:macro>
   <!-- right elbow joint -->
   <xacro:macro name="insert_mesh_r_el_link">
@@ -164,4 +254,10 @@
     </material>
   </xacro:macro>
+  <xacro:macro name="insert_box_r_el_link">
+    <origin xyz="-0.0190 -0.0720 0.0000" rpy="0.0000 -0.0000 -0.0000"/>
+    <geometry>
+      <box size="0.0420 0.1490 0.0300"/>
+    </geometry>
+  </xacro:macro>
   <!-- left shoulder pitch joint -->
   <xacro:macro name="insert_mesh_l_sho_pitch_link">
@@ -174,4 +270,10 @@
     </material>
   </xacro:macro>
+  <xacro:macro name="insert_box_l_sho_pitch_link">
+    <origin xyz="0.0000 0.0155 -0.0038" rpy="0.0000 -0.0000 -0.0000"/>
+    <geometry>
+      <box size="0.0420 0.0310 0.0325"/>
+    </geometry>
+  </xacro:macro>
   <!-- left shoulder pitch joint -->
   <xacro:macro name="insert_mesh_l_sho_roll_link">
@@ -184,4 +286,10 @@
     </material>
   </xacro:macro>
+  <xacro:macro name="insert_box_l_sho_roll_link">
+    <origin xyz="-0.0168 0.0452 0.0007" rpy="0.0000 -0.0000 -0.0000"/>
+    <geometry>
+      <box size="0.0424 0.1129 0.0301"/>
+    </geometry>
+  </xacro:macro>
   <!-- left elbow joint -->
   <xacro:macro name="insert_mesh_l_el_link">
@@ -194,4 +302,10 @@
     </material>
   </xacro:macro>
+  <xacro:macro name="insert_box_l_el_link">
+    <origin xyz="-0.0190 0.0720 0.0000" rpy="0.0000 -0.0000 -0.0000"/>
+    <geometry>
+      <box size="0.0420 0.1490 0.0300"/>
+    </geometry>
+  </xacro:macro>
   <!-- head yaw joint -->
   <xacro:macro name="insert_mesh_head_pan_link">
@@ -204,4 +318,13 @@
     </material>
   </xacro:macro>
+  <xacro:macro name="insert_box_head_pan_link">
+    <origin xyz="0.0038 -0.0000 0.0155" rpy="0.0000 -0.0000 -0.0000"/>
+    <geometry>
+      <box size="0.0325 0.0420 0.0310"/>
+    </geometry>
+    <material name="Grey">
+      <color rgba="0.60 0.60 0.60 1.0"/>
+    </material>
+  </xacro:macro>
   <!-- head yaw joint -->
   <xacro:macro name="insert_mesh_head_tilt_link">
@@ -214,3 +337,9 @@
     </material>
   </xacro:macro>
+  <xacro:macro name="insert_box_head_tilt_link">
+    <origin xyz="0.0060 -0.0190 0.0278" rpy="0.0000 -0.0000 -0.0000"/>
+    <geometry>
+      <box size="0.0445 0.0940 0.0780"/>
+    </geometry>
+  </xacro:macro>
 </robot>

Commit message: Fix motor specs

File: op3_description/urdf/robotis_op3.structure.head.xacro (robot description, xacro)
@@ -12,5 +12,5 @@
       <origin xyz="-0.001 0.0 0.1365" rpy="0 0 0"/>
       <axis xyz="0 0 1"/>
-      <limit effort="1000" velocity="100" lower="${-pi*0.9}" upper="${pi*0.9}"/>
+      <limit effort="3.40" velocity="3.14" lower="${-pi*0.9}" upper="${pi*0.9}"/>
       <dynamics damping="0.0" friction="0.1"/>
     </joint>
@@ -34,5 +34,5 @@
       <origin xyz="0.010 0.019 0.0285" rpy="0 0 0"/>
       <axis xyz="0 -1 0"/>
-      <limit effort="1000" velocity="100" lower="${-pi*0.9}" upper="${pi*0.9}"/>
+      <limit effort="3.40" velocity="3.14" lower="${-pi*0.9}" upper="${pi*0.9}"/>
       <dynamics damping="0.0" friction="0.1"/>
     </joint>

File: op3_description/urdf/robotis_op3.structure.larm.xacro (robot description, xacro)
@@ -12,5 +12,5 @@
       <origin xyz="-0.001 0.06 0.111" rpy="0 0 0"/>
       <axis xyz="0 1 0"/>
-      <limit effort="1000" velocity="100" lower="${-pi*0.9}" upper="${pi*0.9}"/>
+      <limit effort="3.40" velocity="3.14" lower="${-pi*0.9}" upper="${pi*0.9}"/>
       <dynamics damping="0.0" friction="0.1"/>
     </joint>
@@ -34,5 +34,5 @@
       <origin xyz="0.019 0.0285 -0.010" rpy="0 0 0"/>
       <axis xyz="-1 0 0"/>
-      <limit effort="1000" velocity="100" lower="${-pi*0.9}" upper="${pi*0.9}"/>
+      <limit effort="3.40" velocity="3.14" lower="${-pi*0.9}" upper="${pi*0.9}"/>
       <dynamics damping="0.0" friction="0.1"/>
     </joint>
@@ -56,5 +56,5 @@
       <origin xyz="0.0 0.0904 -0.0001" rpy="0 0 0"/>
       <axis xyz="1 0 0"/>
-      <limit effort="1000" velocity="100" lower="${-pi*0.9}" upper="${pi*0.9}"/>
+      <limit effort="3.40" velocity="3.14" lower="${-pi*0.9}" upper="${pi*0.9}"/>
       <dynamics damping="0.0" friction="0.1"/>
     </joint>

File: op3_description/urdf/robotis_op3.structure.lleg.xacro (robot description, xacro)
@@ -12,5 +12,5 @@
       <origin xyz="0.0 0.035 0.0" rpy="0 0 0"/>
       <axis xyz="0 0 -1"/>
-      <limit effort="1000" velocity="100" lower="${-pi*0.9}" upper="${pi*0.9}"/>
+      <limit effort="3.40" velocity="3.14" lower="${-pi*0.9}" upper="${pi*0.9}"/>
       <dynamics damping="0.0" friction="0.1"/>
     </joint>
@@ -34,5 +34,5 @@
       <origin xyz="-0.024 0.0 -0.0285" rpy="0 0 0"/>
       <axis xyz="-1 0 0"/>
-      <limit effort="1000" velocity="100" lower="${-pi*0.9}" upper="${pi*0.9}"/>
+      <limit effort="3.40" velocity="3.14" lower="${-pi*0.9}" upper="${pi*0.9}"/>
       <dynamics damping="0.0" friction="0.1"/>
     </joint>
@@ -56,5 +56,5 @@
       <origin xyz="0.0241 0.019 0.0" rpy="0 0 0"/>
       <axis xyz="0 1 0"/>
-      <limit effort="1000" velocity="100" lower="${-pi*0.9}" upper="${pi*0.9}"/>
+      <limit effort="3.40" velocity="3.14" lower="${-pi*0.9}" upper="${pi*0.9}"/>
       <dynamics damping="0.0" friction="0.1"/>
     </joint>
@@ -78,5 +78,5 @@
       <origin xyz="0.0 0.0 -0.11015" rpy="0 0 0"/>
       <axis xyz="0 1 0"/>
-      <limit effort="1000" velocity="100" lower="${-pi*0.9}" upper="${pi*0.9}"/>
+      <limit effort="3.40" velocity="3.14" lower="${-pi*0.9}" upper="${pi*0.9}"/>
       <dynamics damping="0.0" friction="0.1"/>
     </joint>
@@ -100,5 +100,5 @@
       <origin xyz="0 0 -0.110" rpy="0 0 0"/>
       <axis xyz="0 -1 0"/>
-      <limit effort="1000" velocity="100" lower="${-pi*0.9}" upper="${pi*0.9}"/>
+      <limit effort="3.40" velocity="3.14" lower="${-pi*0.9}" upper="${pi*0.9}"/>
       <dynamics damping="0.0" friction="0.1"/>
     </joint>
@@ -122,5 +122,5 @@
       <origin xyz="-0.0241 -0.019 0" rpy="0 0 0"/>
       <axis xyz="1 0 0"/>
-      <limit effort="1000" velocity="100" lower="${-pi*0.9}" upper="${pi*0.9}"/>
+      <limit effort="3.40" velocity="3.14" lower="${-pi*0.9}" upper="${pi*0.9}"/>
       <dynamics damping="0.0" friction="0.1"/>
     </joint>

File: op3_description/urdf/robotis_op3.structure.rarm.xacro (robot description, xacro)
@@ -12,5 +12,5 @@
       <origin xyz="-0.001 -0.06 0.111" rpy="0 0 0"/>
       <axis xyz="0 -1 0"/>
-      <limit effort="1000" velocity="100" lower="${-pi*0.9}" upper="${pi*0.9}"/>
+      <limit effort="3.40" velocity="3.14" lower="${-pi*0.9}" upper="${pi*0.9}"/>
       <dynamics damping="0.0" friction="0.1"/>
     </joint>
@@ -34,5 +34,5 @@
       <origin xyz="0.019 -0.0285 -0.010" rpy="0 0 0"/>
       <axis xyz="-1 0 0"/>
-      <limit effort="1000" velocity="100" lower="${-pi*0.9}" upper="${pi*0.9}"/>
+      <limit effort="3.40" velocity="3.14" lower="${-pi*0.9}" upper="${pi*0.9}"/>
       <dynamics damping="0.0" friction="0.1"/>
     </joint>
@@ -56,5 +56,5 @@
       <origin xyz="0.0 -0.0904 -0.0001" rpy="0 0 0"/>
       <axis xyz="1 0 0"/>
-      <limit effort="1000" velocity="100" lower="${-pi*0.9}" upper="${pi*0.9}"/>
+      <limit effort="3.40" velocity="3.14" lower="${-pi*0.9}" upper="${pi*0.9}"/>
       <dynamics damping="0.0" friction="0.1"/>
     </joint>

File: op3_description/urdf/robotis_op3.structure.rleg.xacro (robot description, xacro)
@@ -12,5 +12,5 @@
       <origin xyz="0.0 -0.035 0.0" rpy="0 0 0"/>
       <axis xyz="0 0 -1"/>
-      <limit effort="1000" velocity="100" lower="${-pi*0.9}" upper="${pi*0.9}"/>
+      <limit effort="3.40" velocity="3.14" lower="${-pi*0.9}" upper="${pi*0.9}"/>
       <dynamics damping="0.0" friction="0.1"/>
     </joint>
@@ -34,5 +34,5 @@
       <origin xyz="-0.024 0.0 -0.0285" rpy="0 0 0"/>
       <axis xyz="-1 0 0"/>
-      <limit effort="1000" velocity="100" lower="${-pi*0.9}" upper="${pi*0.9}"/>
+      <limit effort="3.40" velocity="3.14" lower="${-pi*0.9}" upper="${pi*0.9}"/>
       <dynamics damping="0.0" friction="0.1"/>
     </joint>
@@ -56,5 +56,5 @@
       <origin xyz="0.0241 -0.019 0.0" rpy="0 0 0"/>
       <axis xyz="0 -1 0"/>
-      <limit effort="1000" velocity="100" lower="${-pi*0.9}" upper="${pi*0.9}"/>
+      <limit effort="3.40" velocity="3.14" lower="${-pi*0.9}" upper="${pi*0.9}"/>
       <dynamics damping="0.0" friction="0.1"/>
     </joint>
@@ -78,5 +78,5 @@
       <origin xyz="0.0 0.0 -0.11015" rpy="0 0 0"/>
       <axis xyz="0 -1 0"/>
-      <limit effort="1000" velocity="100" lower="${-pi*0.9}" upper="${pi*0.9}"/>
+      <limit effort="3.40" velocity="3.14" lower="${-pi*0.9}" upper="${pi*0.9}"/>
       <dynamics damping="0.0" friction="0.1"/>
     </joint>
@@ -100,5 +100,5 @@
       <origin xyz="0 0 -0.110" rpy="0 0 0"/>
       <axis xyz="0 1 0"/>
-      <limit effort="1000" velocity="100" lower="${-pi*0.9}" upper="${pi*0.9}"/>
+      <limit effort="3.40" velocity="3.14" lower="${-pi*0.9}" upper="${pi*0.9}"/>
       <dynamics damping="0.0" friction="0.1"/>
     </joint>
@@ -122,5 +122,5 @@
       <origin xyz="-0.0241 0.019 0" rpy="0 0 0"/>
       <axis xyz="1 0 0"/>
-      <limit effort="1000" velocity="100" lower="${-pi*0.9}" upper="${pi*0.9}"/>
+      <limit effort="3.40" velocity="3.14" lower="${-pi*0.9}" upper="${pi*0.9}"/>
       <dynamics damping="0.0" friction="0.1"/>
     </joint>
