Commit message: Fix physics(WIP)

File: op3_description/urdf/gazebo_harness.xacro (robot description, xacro)
@@ -25,7 +25,10 @@
             <ode>
               <implicit_spring_damper>1</implicit_spring_damper>
+              <cfm_damping>0</cfm_damping>
+              <cfm>1e-7</cfm>
+              <erp>0.8</erp>
               <limit>
-                <cfm>0.0</cfm>
-                <erp>0.0</erp>
+                <cfm>1e-7</cfm>
+                <erp>0.8</erp>
               </limit>
             </ode>

File: op3_description/urdf/robotis_op3.gazebo.xacro (robot description, xacro)
@@ -14,5 +14,5 @@
     <minDepth>0.001</minDepth>
     <maxContacts>6</maxContacts>
-    <dampingFactor>0.001</dampingFactor>
+    <dampingFactor>0.0</dampingFactor>
     <selfCollide>false</selfCollide>
     <material>Gazebo/White</material>
@@ -26,5 +26,5 @@
     <minDepth>0.001</minDepth>
     <maxContacts>6</maxContacts>
-    <dampingFactor>0.001</dampingFactor>
+    <dampingFactor>0.0</dampingFactor>
     <selfCollide>false</selfCollide>
     <material>Gazebo/White</material>
@@ -37,5 +37,5 @@
     <minDepth>0.001</minDepth>
     <maxContacts>6</maxContacts>
-    <dampingFactor>0.001</dampingFactor>
+    <dampingFactor>0.0</dampingFactor>
     <selfCollide>false</selfCollide>
     <material>Gazebo/White</material>
@@ -48,5 +48,5 @@
     <minDepth>0.001</minDepth>
     <maxContacts>6</maxContacts>
-    <dampingFactor>0.001</dampingFactor>
+    <dampingFactor>0.0</dampingFactor>
     <selfCollide>false</selfCollide>
     <material>Gazebo/White</material>
@@ -59,5 +59,5 @@
     <minDepth>0.001</minDepth>
     <maxContacts>6</maxContacts>
-    <dampingFactor>0.001</dampingFactor>
+    <dampingFactor>0.0</dampingFactor>
     <selfCollide>false</selfCollide>
     <material>Gazebo/White</material>
@@ -70,5 +70,5 @@
     <minDepth>0.001</minDepth>
     <maxContacts>6</maxContacts>
-    <dampingFactor>0.001</dampingFactor>
+    <dampingFactor>0.0</dampingFactor>
     <selfCollide>false</selfCollide>
     <material>Gazebo/White</material>
@@ -81,5 +81,5 @@
     <minDepth>0.001</minDepth>
     <maxContacts>6</maxContacts>
-    <dampingFactor>0.001</dampingFactor>
+    <dampingFactor>0.0</dampingFactor>
     <material>Gazebo/White</material>
   </gazebo>
@@ -92,5 +92,5 @@
     <minDepth>0.001</minDepth>
     <maxContacts>6</maxContacts>
-    <dampingFactor>0.001</dampingFactor>
+    <dampingFactor>0.0</dampingFactor>
     <selfCollide>false</selfCollide>
     <material>Gazebo/White</material>
@@ -103,5 +103,5 @@
     <minDepth>0.001</minDepth>
     <maxContacts>6</maxContacts>
-    <dampingFactor>0.001</dampingFactor>
+    <dampingFactor>0.0</dampingFactor>
     <selfCollide>false</selfCollide>
     <material>Gazebo/White</material>
@@ -114,5 +114,5 @@
     <minDepth>0.001</minDepth>
     <maxContacts>6</maxContacts>
-    <dampingFactor>0.001</dampingFactor>
+    <dampingFactor>0.0</dampingFactor>
     <selfCollide>false</selfCollide>
     <material>Gazebo/White</material>
@@ -125,5 +125,5 @@
     <minDepth>0.001</minDepth>
     <maxContacts>6</maxContacts>
-    <dampingFactor>0.001</dampingFactor>
+    <dampingFactor>0.0</dampingFactor>
     <selfCollide>false</selfCollide>
     <material>Gazebo/White</material>
@@ -136,5 +136,5 @@
     <minDepth>0.001</minDepth>
     <maxContacts>6</maxContacts>
-    <dampingFactor>0.001</dampingFactor>
+    <dampingFactor>0.0</dampingFactor>
     <selfCollide>false</selfCollide>
     <material>Gazebo/White</material>
@@ -147,5 +147,5 @@
     <minDepth>0.001</minDepth>
     <maxContacts>6</maxContacts>
-    <dampingFactor>0.001</dampingFactor>
+    <dampingFactor>0.0</dampingFactor>
     <selfCollide>false</selfCollide>
     <material>Gazebo/White</material>
@@ -158,5 +158,5 @@
     <minDepth>0.001</minDepth>
     <maxContacts>6</maxContacts>
-    <dampingFactor>0.001</dampingFactor>
+    <dampingFactor>0.0</dampingFactor>
     <selfCollide>false</selfCollide>
     <material>Gazebo/White</material>
@@ -169,5 +169,5 @@
     <minDepth>0.001</minDepth>
     <maxContacts>6</maxContacts>
-    <dampingFactor>0.001</dampingFactor>
+    <dampingFactor>0.0</dampingFactor>
     <selfCollide>false</selfCollide>
     <material>Gazebo/White</material>
@@ -180,5 +180,5 @@
     <minDepth>0.001</minDepth>
     <maxContacts>6</maxContacts>
-    <dampingFactor>0.001</dampingFactor>
+    <dampingFactor>0.0</dampingFactor>
     <selfCollide>false</selfCollide>
     <material>Gazebo/White</material>
@@ -191,5 +191,5 @@
     <minDepth>0.001</minDepth>
     <maxContacts>6</maxContacts>
-    <dampingFactor>0.001</dampingFactor>
+    <dampingFactor>0.0</dampingFactor>
     <selfCollide>false</selfCollide>
     <material>Gazebo/White</material>
@@ -202,5 +202,5 @@
     <minDepth>0.001</minDepth>
     <maxContacts>6</maxContacts>
-    <dampingFactor>0.001</dampingFactor>
+    <dampingFactor>0.0</dampingFactor>
     <selfCollide>false</selfCollide>
     <material>Gazebo/White</material>
@@ -213,5 +213,5 @@
     <minDepth>0.001</minDepth>
     <maxContacts>6</maxContacts>
-    <dampingFactor>0.001</dampingFactor>
+    <dampingFactor>0.0</dampingFactor>
     <selfCollide>false</selfCollide>
     <material>Gazebo/White</material>
@@ -224,5 +224,5 @@
     <minDepth>0.001</minDepth>
     <maxContacts>6</maxContacts>
-    <dampingFactor>0.001</dampingFactor>
+    <dampingFactor>0.0</dampingFactor>
     <selfCollide>false</selfCollide>
     <material>Gazebo/White</material>
@@ -235,5 +235,5 @@
     <minDepth>0.001</minDepth>
     <maxContacts>6</maxContacts>
-    <dampingFactor>0.001</dampingFactor>
+    <dampingFactor>0.0</dampingFactor>
     <selfCollide>false</selfCollide>
     <material>Gazebo/White</material>

File: op3_description/urdf/robotis_op3.structure.head.xacro (robot description, xacro)
@@ -13,5 +13,5 @@
       <axis xyz="0 0 1"/>
       <limit effort="3.40" velocity="3.14" lower="${-pi*0.9}" upper="${pi*0.9}"/>
-      <dynamics damping="0.0" friction="0.1"/>
+      <dynamics damping="1.08" friction="0.0"/>
     </joint>
     <xacro:insert_transmission name="head_pan"/>
@@ -35,5 +35,5 @@
       <axis xyz="0 -1 0"/>
       <limit effort="3.40" velocity="3.14" lower="${-pi*0.9}" upper="${pi*0.9}"/>
-      <dynamics damping="0.0" friction="0.1"/>
+      <dynamics damping="1.08" friction="0.0"/>
     </joint>
     <xacro:insert_transmission name="head_tilt"/>

File: op3_description/urdf/robotis_op3.structure.larm.xacro (robot description, xacro)
@@ -13,5 +13,5 @@
       <axis xyz="0 1 0"/>
       <limit effort="3.40" velocity="3.14" lower="${-pi*0.9}" upper="${pi*0.9}"/>
-      <dynamics damping="0.0" friction="0.1"/>
+      <dynamics damping="1.08" friction="0.0"/>
     </joint>
     <xacro:insert_transmission name="l_sho_pitch"/>
@@ -35,5 +35,5 @@
       <axis xyz="-1 0 0"/>
       <limit effort="3.40" velocity="3.14" lower="${-pi*0.9}" upper="${pi*0.9}"/>
-      <dynamics damping="0.0" friction="0.1"/>
+      <dynamics damping="1.08" friction="0.0"/>
     </joint>
     <xacro:insert_transmission name="l_sho_roll"/>
@@ -57,5 +57,5 @@
       <axis xyz="1 0 0"/>
       <limit effort="3.40" velocity="3.14" lower="${-pi*0.9}" upper="${pi*0.9}"/>
-      <dynamics damping="0.0" friction="0.1"/>
+      <dynamics damping="1.08" friction="0.0"/>
     </joint>
     <xacro:insert_transmission name="l_el"/>

File: op3_description/urdf/robotis_op3.structure.lleg.xacro (robot description, xacro)
@@ -13,5 +13,5 @@
       <axis xyz="0 0 -1"/>
       <limit effort="3.40" velocity="3.14" lower="${-pi*0.9}" upper="${pi*0.9}"/>
-      <dynamics damping="0.0" friction="0.1"/>
+      <dynamics damping="1.08" friction="0.0"/>
     </joint>
     <xacro:insert_transmission name="l_hip_yaw"/>
@@ -35,5 +35,5 @@
       <axis xyz="-1 0 0"/>
       <limit effort="3.40" velocity="3.14" lower="${-pi*0.9}" upper="${pi*0.9}"/>
-      <dynamics damping="0.0" friction="0.1"/>
+      <dynamics damping="1.08" friction="0.0"/>
     </joint>
     <xacro:insert_transmission name="l_hip_roll"/>
@@ -57,5 +57,5 @@
       <axis xyz="0 1 0"/>
       <limit effort="3.40" velocity="3.14" lower="${-pi*0.9}" upper="${pi*0.9}"/>
-      <dynamics damping="0.0" friction="0.1"/>
+      <dynamics damping="1.08" friction="0.0"/>
     </joint>
     <xacro:insert_transmission name="l_hip_pitch"/>
@@ -79,5 +79,5 @@
       <axis xyz="0 1 0"/>
       <limit effort="3.40" velocity="3.14" lower="${-pi*0.9}" upper="${pi*0.9}"/>
-      <dynamics damping="0.0" friction="0.1"/>
+      <dynamics damping="1.08" friction="0.0"/>
     </joint>
     <xacro:insert_transmission name="l_knee"/>
@@ -101,5 +101,5 @@
       <axis xyz="0 -1 0"/>
       <limit effort="3.40" velocity="3.14" lower="${-pi*0.9}" upper="${pi*0.9}"/>
-      <dynamics damping="0.0" friction="0.1"/>
+      <dynamics damping="1.08" friction="0.0"/>
     </joint>
     <xacro:insert_transmission name="l_ank_pitch"/>
@@ -123,5 +123,5 @@
       <axis xyz="1 0 0"/>
       <limit effort="3.40" velocity="3.14" lower="${-pi*0.9}" upper="${pi*0.9}"/>
-      <dynamics damping="0.0" friction="0.1"/>
+      <dynamics damping="1.08" friction="0.0"/>
     </joint>
     <xacro:insert_transmission name="l_ank_roll"/>

File: op3_description/urdf/robotis_op3.structure.rarm.xacro (robot description, xacro)
@@ -13,5 +13,5 @@
       <axis xyz="0 -1 0"/>
       <limit effort="3.40" velocity="3.14" lower="${-pi*0.9}" upper="${pi*0.9}"/>
-      <dynamics damping="0.0" friction="0.1"/>
+      <dynamics damping="1.08" friction="0.0"/>
     </joint>
     <xacro:insert_transmission name="r_sho_pitch"/>
@@ -35,5 +35,5 @@
       <axis xyz="-1 0 0"/>
       <limit effort="3.40" velocity="3.14" lower="${-pi*0.9}" upper="${pi*0.9}"/>
-      <dynamics damping="0.0" friction="0.1"/>
+      <dynamics damping="1.08" friction="0.0"/>
     </joint>
     <xacro:insert_transmission name="r_sho_roll"/>
@@ -57,5 +57,5 @@
       <axis xyz="1 0 0"/>
       <limit effort="3.40" velocity="3.14" lower="${-pi*0.9}" upper="${pi*0.9}"/>
-      <dynamics damping="0.0" friction="0.1"/>
+      <dynamics damping="1.08" friction="0.0"/>
     </joint>
     <xacro:insert_transmission name="r_el"/>

File: op3_description/urdf/robotis_op3.structure.rleg.xacro (robot description, xacro)
@@ -13,5 +13,5 @@
       <axis xyz="0 0 -1"/>
       <limit effort="3.40" velocity="3.14" lower="${-pi*0.9}" upper="${pi*0.9}"/>
-      <dynamics damping="0.0" friction="0.1"/>
+      <dynamics damping="1.08" friction="0.0"/>
     </joint>
     <xacro:insert_transmission name="r_hip_yaw"/>
@@ -35,5 +35,5 @@
       <axis xyz="-1 0 0"/>
       <limit effort="3.40" velocity="3.14" lower="${-pi*0.9}" upper="${pi*0.9}"/>
-      <dynamics damping="0.0" friction="0.1"/>
+      <dynamics damping="1.08" friction="0.0"/>
     </joint>
     <xacro:insert_transmission name="r_hip_roll"/>
@@ -57,5 +57,5 @@
       <axis xyz="0 -1 0"/>
       <limit effort="3.40" velocity="3.14" lower="${-pi*0.9}" upper="${pi*0.9}"/>
-      <dynamics damping="0.0" friction="0.1"/>
+      <dynamics damping="1.08" friction="0.0"/>
     </joint>
     <xacro:insert_transmission name="r_hip_pitch"/>
@@ -79,5 +79,5 @@
       <axis xyz="0 -1 0"/>
       <limit effort="3.40" velocity="3.14" lower="${-pi*0.9}" upper="${pi*0.9}"/>
-      <dynamics damping="0.0" friction="0.1"/>
+      <dynamics damping="1.08" friction="0.0"/>
     </joint>
     <xacro:insert_transmission name="r_knee"/>
@@ -101,5 +101,5 @@
       <axis xyz="0 1 0"/>
       <limit effort="3.40" velocity="3.14" lower="${-pi*0.9}" upper="${pi*0.9}"/>
-      <dynamics damping="0.0" friction="0.1"/>
+      <dynamics damping="1.08" friction="0.0"/>
     </joint>
     <xacro:insert_transmission name="r_ank_pitch"/>
@@ -123,5 +123,5 @@
       <axis xyz="1 0 0"/>
       <limit effort="3.40" velocity="3.14" lower="${-pi*0.9}" upper="${pi*0.9}"/>
-      <dynamics damping="0.0" friction="0.1"/>
+      <dynamics damping="1.08" friction="0.0"/>
     </joint>
     <xacro:insert_transmission name="r_ank_roll"/>
