Commit message: Update physics

File: op3_description/urdf/robotis_op3.gazebo.xacro (robot description, xacro)
@@ -8,222 +8,515 @@
   <!-- body link -->
   <gazebo reference="body_link">
-    <mu1>0.2</mu1>
-    <mu2>0.2</mu2>
-    <material>Gazebo/White</material>
-    <selfCollide>false</selfCollide>
+    <kp>100000.0</kp>
+    <kd>10.0</kd>
+    <mu1>0.1</mu1>
+    <maxVel>10.0</maxVel>
+    <minDepth>0.001</minDepth>
+    <maxContacts>6</maxContacts>
+    <dampingFactor>0.001</dampingFactor>
+    <selfCollide>false</selfCollide>
+    <material>Gazebo/White</material>
   </gazebo>
   <!-- left leg links -->
   <gazebo reference="l_hip_yaw_link">
-    <mu1>0.2</mu1>
-    <mu2>0.2</mu2>
-    <material>Gazebo/White</material>
-    <selfCollide>false</selfCollide>
+    <kp>100000.0</kp>
+    <kd>10.0</kd>
+    <mu1>0.1</mu1>
+    <maxVel>10.0</maxVel>
+    <minDepth>0.001</minDepth>
+    <maxContacts>6</maxContacts>
+    <dampingFactor>0.001</dampingFactor>
+    <selfCollide>false</selfCollide>
+    <material>Gazebo/White</material>
   </gazebo>
   <gazebo reference="l_hip_roll_link">
-    <mu1>0.2</mu1>
-    <mu2>0.2</mu2>
-    <material>Gazebo/White</material>
-    <selfCollide>false</selfCollide>
+    <kp>100000.0</kp>
+    <kd>10.0</kd>
+    <mu1>0.1</mu1>
+    <maxVel>10.0</maxVel>
+    <minDepth>0.001</minDepth>
+    <maxContacts>6</maxContacts>
+    <dampingFactor>0.001</dampingFactor>
+    <selfCollide>false</selfCollide>
+    <material>Gazebo/White</material>
   </gazebo>
   <gazebo reference="l_hip_pitch_link">
-    <mu1>0.2</mu1>
-    <mu2>0.2</mu2>
-    <material>Gazebo/White</material>
-    <selfCollide>false</selfCollide>
+    <kp>100000.0</kp>
+    <kd>10.0</kd>
+    <mu1>0.1</mu1>
+    <maxVel>10.0</maxVel>
+    <minDepth>0.001</minDepth>
+    <maxContacts>6</maxContacts>
+    <dampingFactor>0.001</dampingFactor>
+    <selfCollide>false</selfCollide>
+    <material>Gazebo/White</material>
   </gazebo>
   <gazebo reference="l_knee_link">
-    <mu1>0.2</mu1>
-    <mu2>0.2</mu2>
-    <material>Gazebo/White</material>
-    <selfCollide>false</selfCollide>
+    <kp>100000.0</kp>
+    <kd>10.0</kd>
+    <mu1>0.1</mu1>
+    <maxVel>10.0</maxVel>
+    <minDepth>0.001</minDepth>
+    <maxContacts>6</maxContacts>
+    <dampingFactor>0.001</dampingFactor>
+    <selfCollide>false</selfCollide>
+    <material>Gazebo/White</material>
   </gazebo>
   <gazebo reference="l_ank_pitch_link">
-    <mu1>0.2</mu1>
-    <mu2>0.2</mu2>
-    <material>Gazebo/White</material>
-    <selfCollide>false</selfCollide>
+    <kp>100000.0</kp>
+    <kd>10.0</kd>
+    <mu1>0.1</mu1>
+    <maxVel>10.0</maxVel>
+    <minDepth>0.001</minDepth>
+    <maxContacts>6</maxContacts>
+    <dampingFactor>0.001</dampingFactor>
+    <selfCollide>false</selfCollide>
+    <material>Gazebo/White</material>
   </gazebo>
   <gazebo reference="l_ank_roll_link">
     <kp>100000.0</kp>
-    <kd>100.0</kd>
-    <mu1>1.5</mu1>
-    <mu2>1.5</mu2>
-    <fdir1>1 0 0</fdir1>
-    <maxVel>1.0</maxVel>
-    <minDepth>0.001</minDepth>
+    <kd>10.0</kd>
+    <mu1>1.0</mu1>
+    <maxVel>10.0</maxVel>
+    <minDepth>0.001</minDepth>
+    <maxContacts>6</maxContacts>
+    <dampingFactor>0.001</dampingFactor>
     <material>Gazebo/White</material>
   </gazebo>
   <!-- right leg links -->
   <gazebo reference="r_hip_yaw_link">
-    <mu1>0.2</mu1>
-    <mu2>0.2</mu2>
-    <material>Gazebo/White</material>
-    <selfCollide>false</selfCollide>
+    <kp>100000.0</kp>
+    <kd>10.0</kd>
+    <mu1>0.1</mu1>
+    <maxVel>10.0</maxVel>
+    <minDepth>0.001</minDepth>
+    <maxContacts>6</maxContacts>
+    <dampingFactor>0.001</dampingFactor>
+    <selfCollide>false</selfCollide>
+    <material>Gazebo/White</material>
   </gazebo>
   <gazebo reference="r_hip_roll_link">
-    <mu1>0.2</mu1>
-    <mu2>0.2</mu2>
-    <material>Gazebo/White</material>
-    <selfCollide>false</selfCollide>
+    <kp>100000.0</kp>
+    <kd>10.0</kd>
+    <mu1>0.1</mu1>
+    <maxVel>10.0</maxVel>
+    <minDepth>0.001</minDepth>
+    <maxContacts>6</maxContacts>
+    <dampingFactor>0.001</dampingFactor>
+    <selfCollide>false</selfCollide>
+    <material>Gazebo/White</material>
   </gazebo>
   <gazebo reference="r_hip_pitch_link">
-    <mu1>0.2</mu1>
-    <mu2>0.2</mu2>
-    <material>Gazebo/White</material>
-    <selfCollide>false</selfCollide>
+    <kp>100000.0</kp>
+    <kd>10.0</kd>
+    <mu1>0.1</mu1>
+    <maxVel>10.0</maxVel>
+    <minDepth>0.001</minDepth>
+    <maxContacts>6</maxContacts>
+    <dampingFactor>0.001</dampingFactor>
+    <selfCollide>false</selfCollide>
+    <material>Gazebo/White</material>
   </gazebo>
   <gazebo reference="r_knee_link">
-    <mu1>0.2</mu1>
-    <mu2>0.2</mu2>
-    <material>Gazebo/White</material>
-    <selfCollide>false</selfCollide>
+    <kp>100000.0</kp>
+    <kd>10.0</kd>
+    <mu1>0.1</mu1>
+    <maxVel>10.0</maxVel>
+    <minDepth>0.001</minDepth>
+    <maxContacts>6</maxContacts>
+    <dampingFactor>0.001</dampingFactor>
+    <selfCollide>false</selfCollide>
+    <material>Gazebo/White</material>
   </gazebo>
   <gazebo reference="r_ank_pitch_link">
-    <mu1>0.2</mu1>
-    <mu2>0.2</mu2>
-    <material>Gazebo/White</material>
-    <selfCollide>false</selfCollide>
+    <kp>100000.0</kp>
+    <kd>10.0</kd>
+    <mu1>0.1</mu1>
+    <maxVel>10.0</maxVel>
+    <minDepth>0.001</minDepth>
+    <maxContacts>6</maxContacts>
+    <dampingFactor>0.001</dampingFactor>
+    <selfCollide>false</selfCollide>
+    <material>Gazebo/White</material>
   </gazebo>
   <gazebo reference="r_ank_roll_link">
-    <mu1>9000</mu1>
-    <kp>100000.0</kp>
-    <kd>100.0</kd>
-    <mu1>1.5</mu1>
-    <mu2>1.5</mu2>
-    <fdir1>1 0 0</fdir1>
-    <maxVel>1.0</maxVel>
-    <minDepth>0.001</minDepth>
+    <kp>100000.0</kp>
+    <kd>10.0</kd>
+    <mu1>1.0</mu1>
+    <maxVel>10.0</maxVel>
+    <minDepth>0.001</minDepth>
+    <maxContacts>6</maxContacts>
+    <dampingFactor>0.001</dampingFactor>
+    <selfCollide>false</selfCollide>
     <material>Gazebo/White</material>
   </gazebo>
   <gazebo reference="r_sho_pitch_link">
-    <mu1>0.2</mu1>
-    <mu2>0.2</mu2>
-    <material>Gazebo/White</material>
-    <selfCollide>false</selfCollide>
+    <kp>100000.0</kp>
+    <kd>10.0</kd>
+    <mu1>0.1</mu1>
+    <maxVel>10.0</maxVel>
+    <minDepth>0.001</minDepth>
+    <maxContacts>6</maxContacts>
+    <dampingFactor>0.001</dampingFactor>
+    <selfCollide>false</selfCollide>
+    <material>Gazebo/White</material>
   </gazebo>
   <gazebo reference="r_sho_roll_link">
-    <mu1>0.2</mu1>
-    <mu2>0.2</mu2>
-    <material>Gazebo/White</material>
-    <selfCollide>false</selfCollide>
+    <kp>100000.0</kp>
+    <kd>10.0</kd>
+    <mu1>0.1</mu1>
+    <maxVel>10.0</maxVel>
+    <minDepth>0.001</minDepth>
+    <maxContacts>6</maxContacts>
+    <dampingFactor>0.001</dampingFactor>
+    <selfCollide>false</selfCollide>
+    <material>Gazebo/White</material>
   </gazebo>
   <gazebo reference="r_el_link">
-    <mu1>0.2</mu1>
-    <mu2>0.2</mu2>
-    <material>Gazebo/White</material>
-    <selfCollide>false</selfCollide>
+    <kp>100000.0</kp>
+    <kd>10.0</kd>
+    <mu1>0.1</mu1>
+    <maxVel>10.0</maxVel>
+    <minDepth>0.001</minDepth>
+    <maxContacts>6</maxContacts>
+    <dampingFactor>0.001</dampingFactor>
+    <selfCollide>false</selfCollide>
+    <material>Gazebo/White</material>
   </gazebo>
   <gazebo reference="l_sho_pitch_link">
-    <mu1>0.2</mu1>
-    <mu2>0.2</mu2>
-    <material>Gazebo/White</material>
-    <selfCollide>false</selfCollide>
+    <kp>100000.0</kp>
+    <kd>10.0</kd>
+    <mu1>0.1</mu1>
+    <maxVel>10.0</maxVel>
+    <minDepth>0.001</minDepth>
+    <maxContacts>6</maxContacts>
+    <dampingFactor>0.001</dampingFactor>
+    <selfCollide>false</selfCollide>
+    <material>Gazebo/White</material>
   </gazebo>
   <gazebo reference="l_sho_roll_link">
-    <mu1>0.2</mu1>
-    <mu2>0.2</mu2>
-    <material>Gazebo/White</material>
-    <selfCollide>false</selfCollide>
+    <kp>100000.0</kp>
+    <kd>10.0</kd>
+    <mu1>0.1</mu1>
+    <maxVel>10.0</maxVel>
+    <minDepth>0.001</minDepth>
+    <maxContacts>6</maxContacts>
+    <dampingFactor>0.001</dampingFactor>
+    <selfCollide>false</selfCollide>
+    <material>Gazebo/White</material>
   </gazebo>
   <gazebo reference="l_el_link">
-    <mu1>0.2</mu1>
-    <mu2>0.2</mu2>
-    <material>Gazebo/White</material>
-    <selfCollide>false</selfCollide>
+    <kp>100000.0</kp>
+    <kd>10.0</kd>
+    <mu1>0.1</mu1>
+    <maxVel>10.0</maxVel>
+    <minDepth>0.001</minDepth>
+    <maxContacts>6</maxContacts>
+    <dampingFactor>0.001</dampingFactor>
+    <selfCollide>false</selfCollide>
+    <material>Gazebo/White</material>
   </gazebo>
   <gazebo reference="head_pan_link">
-    <mu1>0.2</mu1>
-    <mu2>0.2</mu2>
-    <material>Gazebo/White</material>
-    <selfCollide>false</selfCollide>
+    <kp>100000.0</kp>
+    <kd>10.0</kd>
+    <mu1>0.1</mu1>
+    <maxVel>10.0</maxVel>
+    <minDepth>0.001</minDepth>
+    <maxContacts>6</maxContacts>
+    <dampingFactor>0.001</dampingFactor>
+    <selfCollide>false</selfCollide>
+    <material>Gazebo/White</material>
   </gazebo>
   <gazebo reference="head_tilt_link">
-    <mu1>0.2</mu1>
-    <mu2>0.2</mu2>
-    <material>Gazebo/White</material>
-    <selfCollide>false</selfCollide>
-  </gazebo>
-  <!--
+    <kp>100000.0</kp>
+    <kd>10.0</kd>
+    <mu1>0.1</mu1>
+    <maxVel>10.0</maxVel>
+    <minDepth>0.001</minDepth>
+    <maxContacts>6</maxContacts>
+    <dampingFactor>0.001</dampingFactor>
+    <selfCollide>false</selfCollide>
+    <material>Gazebo/White</material>
+  </gazebo>
   <gazebo reference="l_hip_yaw">
-    <provideFeedback>1</provideFeedback>
-    <implicitSpringDamper>1</implicitSpringDamper>
+    <physics>
+      <ode>
+        <implicit_spring_damper>1</implicit_spring_damper>
+        <cfm_damping>0</cfm_damping>
+        <cfm>1e-7</cfm>
+        <erp>0.8</erp>
+        <limit>
+          <cfm>1e-7</cfm>
+          <erp>0.8</erp>
+        </limit>
+      </ode>
+    </physics>
   </gazebo>
   <gazebo reference="l_hip_roll">
-    <provideFeedback>1</provideFeedback>
-    <implicitSpringDamper>1</implicitSpringDamper>
+    <physics>
+      <ode>
+        <implicit_spring_damper>1</implicit_spring_damper>
+        <cfm_damping>0</cfm_damping>
+        <cfm>1e-7</cfm>
+        <erp>0.8</erp>
+        <limit>
+          <cfm>1e-7</cfm>
+          <erp>0.8</erp>
+        </limit>
+      </ode>
+    </physics>
   </gazebo>
   <gazebo reference="l_hip_pitch">
-    <provideFeedback>1</provideFeedback>
-    <implicitSpringDamper>1</implicitSpringDamper>
+    <physics>
+      <ode>
+        <implicit_spring_damper>1</implicit_spring_damper>
+        <cfm_damping>0</cfm_damping>
+        <cfm>1e-7</cfm>
+        <erp>0.8</erp>
+        <limit>
+          <cfm>1e-7</cfm>
+          <erp>0.8</erp>
+        </limit>
+      </ode>
+    </physics>
   </gazebo>
   <gazebo reference="l_knee">
-    <provideFeedback>1</provideFeedback>
-    <implicitSpringDamper>1</implicitSpringDamper>
+    <physics>
+      <ode>
+        <implicit_spring_damper>1</implicit_spring_damper>
+        <cfm_damping>0</cfm_damping>
+        <cfm>1e-7</cfm>
+        <erp>0.8</erp>
+        <limit>
+          <cfm>1e-7</cfm>
+          <erp>0.8</erp>
+        </limit>
+      </ode>
+    </physics>
   </gazebo>
   <gazebo reference="l_ank_roll">
-    <provideFeedback>1</provideFeedback>
-    <implicitSpringDamper>1</implicitSpringDamper>
+    <physics>
+      <ode>
+        <implicit_spring_damper>1</implicit_spring_damper>
+        <cfm_damping>0</cfm_damping>
+        <cfm>1e-7</cfm>
+        <erp>0.8</erp>
+        <limit>
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
File: op3_description/urdf/robotis_op3.structure.head.xacro (robot description, xacro)
@@ -13,5 +13,5 @@
       <axis xyz="0 0 1"/>
       <limit effort="1000" velocity="100" lower="${-pi*0.9}" upper="${pi*0.9}"/>
-      <dynamics damping="0.1" friction="0.0"/>
+      <dynamics damping="0.0" friction="0.1"/>
     </joint>
     <xacro:insert_transmission name="head_pan"/>
@@ -35,5 +35,5 @@
       <axis xyz="0 -1 0"/>
       <limit effort="1000" velocity="100" lower="${-pi*0.9}" upper="${pi*0.9}"/>
-      <dynamics damping="0.1" friction="0.0"/>
+      <dynamics damping="0.0" friction="0.1"/>
     </joint>
     <xacro:insert_transmission name="head_tilt"/>

File: op3_description/urdf/robotis_op3.structure.larm.xacro (robot description, xacro)
@@ -13,5 +13,5 @@
       <axis xyz="0 1 0"/>
       <limit effort="1000" velocity="100" lower="${-pi*0.9}" upper="${pi*0.9}"/>
-      <dynamics damping="0.1" friction="0.0"/>
+      <dynamics damping="0.0" friction="0.1"/>
     </joint>
     <xacro:insert_transmission name="l_sho_pitch"/>
@@ -35,5 +35,5 @@
       <axis xyz="-1 0 0"/>
       <limit effort="1000" velocity="100" lower="${-pi*0.9}" upper="${pi*0.9}"/>
-      <dynamics damping="0.1" friction="0.0"/>
+      <dynamics damping="0.0" friction="0.1"/>
     </joint>
     <xacro:insert_transmission name="l_sho_roll"/>
@@ -57,5 +57,5 @@
       <axis xyz="1 0 0"/>
       <limit effort="1000" velocity="100" lower="${-pi*0.9}" upper="${pi*0.9}"/>
-      <dynamics damping="0.1" friction="0.0"/>
+      <dynamics damping="0.0" friction="0.1"/>
     </joint>
     <xacro:insert_transmission name="l_el"/>

File: op3_description/urdf/robotis_op3.structure.lleg.xacro (robot description, xacro)
@@ -13,5 +13,5 @@
       <axis xyz="0 0 -1"/>
       <limit effort="1000" velocity="100" lower="${-pi*0.9}" upper="${pi*0.9}"/>
-      <dynamics damping="0.1" friction="0.0"/>
+      <dynamics damping="0.0" friction="0.1"/>
     </joint>
     <xacro:insert_transmission name="l_hip_yaw"/>
@@ -35,5 +35,5 @@
       <axis xyz="-1 0 0"/>
       <limit effort="1000" velocity="100" lower="${-pi*0.9}" upper="${pi*0.9}"/>
-      <dynamics damping="0.1" friction="0.0"/>
+      <dynamics damping="0.0" friction="0.1"/>
     </joint>
     <xacro:insert_transmission name="l_hip_roll"/>
@@ -57,5 +57,5 @@
       <axis xyz="0 1 0"/>
       <limit effort="1000" velocity="100" lower="${-pi*0.9}" upper="${pi*0.9}"/>
-      <dynamics damping="0.1" friction="0.0"/>
+      <dynamics damping="0.0" friction="0.1"/>
     </joint>
     <xacro:insert_transmission name="l_hip_pitch"/>
@@ -79,5 +79,5 @@
       <axis xyz="0 1 0"/>
       <limit effort="1000" velocity="100" lower="${-pi*0.9}" upper="${pi*0.9}"/>
-      <dynamics damping="0.1" friction="0.0"/>
+      <dynamics damping="0.0" friction="0.1"/>
     </joint>
     <xacro:insert_transmission name="l_knee"/>
@@ -101,5 +101,5 @@
       <axis xyz="0 -1 0"/>
       <limit effort="1000" velocity="100" lower="${-pi*0.9}" upper="${pi*0.9}"/>
-      <dynamics damping="0.1" friction="0.0"/>
+      <dynamics damping="0.0" friction="0.1"/>
     </joint>
     <xacro:insert_transmission name="l_ank_pitch"/>
@@ -123,5 +123,5 @@
       <axis xyz="1 0 0"/>
       <limit effort="1000" velocity="100" lower="${-pi*0.9}" upper="${pi*0.9}"/>
-      <dynamics damping="0.1" friction="0.0"/>
+      <dynamics damping="0.0" friction="0.1"/>
     </joint>
     <xacro:insert_transmission name="l_ank_roll"/>

File: op3_description/urdf/robotis_op3.structure.rarm.xacro (robot description, xacro)
@@ -13,5 +13,5 @@
       <axis xyz="0 -1 0"/>
       <limit effort="1000" velocity="100" lower="${-pi*0.9}" upper="${pi*0.9}"/>
-      <dynamics damping="0.1" friction="0.0"/>
+      <dynamics damping="0.0" friction="0.1"/>
     </joint>
     <xacro:insert_transmission name="r_sho_pitch"/>
@@ -35,5 +35,5 @@
       <axis xyz="-1 0 0"/>
       <limit effort="1000" velocity="100" lower="${-pi*0.9}" upper="${pi*0.9}"/>
-      <dynamics damping="0.1" friction="0.0"/>
+      <dynamics damping="0.0" friction="0.1"/>
     </joint>
     <xacro:insert_transmission name="r_sho_roll"/>
@@ -57,5 +57,5 @@
       <axis xyz="1 0 0"/>
       <limit effort="1000" velocity="100" lower="${-pi*0.9}" upper="${pi*0.9}"/>
-      <dynamics damping="0.1" friction="0.0"/>
+      <dynamics damping="0.0" friction="0.1"/>
     </joint>
     <xacro:insert_transmission name="r_el"/>

File: op3_description/urdf/robotis_op3.structure.rleg.xacro (robot description, xacro)
@@ -13,5 +13,5 @@
       <axis xyz="0 0 -1"/>
       <limit effort="1000" velocity="100" lower="${-pi*0.9}" upper="${pi*0.9}"/>
-      <dynamics damping="0.1" friction="0.0"/>
+      <dynamics damping="0.0" friction="0.1"/>
     </joint>
     <xacro:insert_transmission name="r_hip_yaw"/>
@@ -35,5 +35,5 @@
       <axis xyz="-1 0 0"/>
       <limit effort="1000" velocity="100" lower="${-pi*0.9}" upper="${pi*0.9}"/>
-      <dynamics damping="0.1" friction="0.0"/>
+      <dynamics damping="0.0" friction="0.1"/>
     </joint>
     <xacro:insert_transmission name="r_hip_roll"/>
@@ -57,5 +57,5 @@
       <axis xyz="0 -1 0"/>
       <limit effort="1000" velocity="100" lower="${-pi*0.9}" upper="${pi*0.9}"/>
-      <dynamics damping="0.1" friction="0.0"/>
+      <dynamics damping="0.0" friction="0.1"/>
     </joint>
     <xacro:insert_transmission name="r_hip_pitch"/>
@@ -79,5 +79,5 @@
       <axis xyz="0 -1 0"/>
       <limit effort="1000" velocity="100" lower="${-pi*0.9}" upper="${pi*0.9}"/>
-      <dynamics damping="0.1" friction="0.0"/>
+      <dynamics damping="0.0" friction="0.1"/>
     </joint>
     <xacro:insert_transmission name="r_knee"/>
@@ -101,5 +101,5 @@
       <axis xyz="0 1 0"/>
       <limit effort="1000" velocity="100" lower="${-pi*0.9}" upper="${pi*0.9}"/>
-      <dynamics damping="0.1" friction="0.0"/>
+      <dynamics damping="0.0" friction="0.1"/>
     </joint>
     <xacro:insert_transmission name="r_ank_pitch"/>
@@ -123,5 +123,5 @@
       <axis xyz="1 0 0"/>
       <limit effort="1000" velocity="100" lower="${-pi*0.9}" upper="${pi*0.9}"/>
-      <dynamics damping="0.1" friction="0.0"/>
+      <dynamics damping="0.0" friction="0.1"/>
     </joint>
     <xacro:insert_transmission name="r_ank_roll"/>
