Commit message: Fix physics(WIP)

File: op3_description/urdf/robotis_op3.gazebo.xacro (robot description, xacro)
@@ -8,9 +8,9 @@
   <!-- body link -->
   <gazebo reference="body_link">
-    <kp>100000.0</kp>
-    <kd>10.0</kd>
-    <mu1>0.1</mu1>
-    <maxVel>10.0</maxVel>
-    <minDepth>0.001</minDepth>
+    <kp>1000000.0</kp>
+    <kd>100.0</kd>
+    <mu1>0.1</mu1>
+    <maxVel>10.0</maxVel>
+    <minDepth>0.0001</minDepth>
     <maxContacts>6</maxContacts>
     <dampingFactor>0.0</dampingFactor>
@@ -20,9 +20,9 @@
   <!-- left leg links -->
   <gazebo reference="l_hip_yaw_link">
-    <kp>100000.0</kp>
-    <kd>10.0</kd>
-    <mu1>0.1</mu1>
-    <maxVel>10.0</maxVel>
-    <minDepth>0.001</minDepth>
+    <kp>1000000.0</kp>
+    <kd>100.0</kd>
+    <mu1>0.1</mu1>
+    <maxVel>10.0</maxVel>
+    <minDepth>0.0001</minDepth>
     <maxContacts>6</maxContacts>
     <dampingFactor>0.0</dampingFactor>
@@ -31,9 +31,9 @@
   </gazebo>
   <gazebo reference="l_hip_roll_link">
-    <kp>100000.0</kp>
-    <kd>10.0</kd>
-    <mu1>0.1</mu1>
-    <maxVel>10.0</maxVel>
-    <minDepth>0.001</minDepth>
+    <kp>1000000.0</kp>
+    <kd>100.0</kd>
+    <mu1>0.1</mu1>
+    <maxVel>10.0</maxVel>
+    <minDepth>0.0001</minDepth>
     <maxContacts>6</maxContacts>
     <dampingFactor>0.0</dampingFactor>
@@ -42,9 +42,9 @@
   </gazebo>
   <gazebo reference="l_hip_pitch_link">
-    <kp>100000.0</kp>
-    <kd>10.0</kd>
-    <mu1>0.1</mu1>
-    <maxVel>10.0</maxVel>
-    <minDepth>0.001</minDepth>
+    <kp>1000000.0</kp>
+    <kd>100.0</kd>
+    <mu1>0.1</mu1>
+    <maxVel>10.0</maxVel>
+    <minDepth>0.0001</minDepth>
     <maxContacts>6</maxContacts>
     <dampingFactor>0.0</dampingFactor>
@@ -53,9 +53,9 @@
   </gazebo>
   <gazebo reference="l_knee_link">
-    <kp>100000.0</kp>
-    <kd>10.0</kd>
-    <mu1>0.1</mu1>
-    <maxVel>10.0</maxVel>
-    <minDepth>0.001</minDepth>
+    <kp>1000000.0</kp>
+    <kd>100.0</kd>
+    <mu1>0.1</mu1>
+    <maxVel>10.0</maxVel>
+    <minDepth>0.0001</minDepth>
     <maxContacts>6</maxContacts>
     <dampingFactor>0.0</dampingFactor>
@@ -64,9 +64,9 @@
   </gazebo>
   <gazebo reference="l_ank_pitch_link">
-    <kp>100000.0</kp>
-    <kd>10.0</kd>
-    <mu1>0.1</mu1>
-    <maxVel>10.0</maxVel>
-    <minDepth>0.001</minDepth>
+    <kp>1000000.0</kp>
+    <kd>100.0</kd>
+    <mu1>0.1</mu1>
+    <maxVel>10.0</maxVel>
+    <minDepth>0.0001</minDepth>
     <maxContacts>6</maxContacts>
     <dampingFactor>0.0</dampingFactor>
@@ -75,9 +75,9 @@
   </gazebo>
   <gazebo reference="l_ank_roll_link">
-    <kp>100000.0</kp>
-    <kd>10.0</kd>
+    <kp>1000000.0</kp>
+    <kd>100.0</kd>
     <mu1>1.0</mu1>
     <maxVel>10.0</maxVel>
-    <minDepth>0.001</minDepth>
+    <minDepth>0.0001</minDepth>
     <maxContacts>6</maxContacts>
     <dampingFactor>0.0</dampingFactor>
@@ -86,9 +86,9 @@
   <!-- right leg links -->
   <gazebo reference="r_hip_yaw_link">
-    <kp>100000.0</kp>
-    <kd>10.0</kd>
-    <mu1>0.1</mu1>
-    <maxVel>10.0</maxVel>
-    <minDepth>0.001</minDepth>
+    <kp>1000000.0</kp>
+    <kd>100.0</kd>
+    <mu1>0.1</mu1>
+    <maxVel>10.0</maxVel>
+    <minDepth>0.0001</minDepth>
     <maxContacts>6</maxContacts>
     <dampingFactor>0.0</dampingFactor>
@@ -97,9 +97,9 @@
   </gazebo>
   <gazebo reference="r_hip_roll_link">
-    <kp>100000.0</kp>
-    <kd>10.0</kd>
-    <mu1>0.1</mu1>
-    <maxVel>10.0</maxVel>
-    <minDepth>0.001</minDepth>
+    <kp>1000000.0</kp>
+    <kd>100.0</kd>
+    <mu1>0.1</mu1>
+    <maxVel>10.0</maxVel>
+    <minDepth>0.0001</minDepth>
     <maxContacts>6</maxContacts>
     <dampingFactor>0.0</dampingFactor>
@@ -108,9 +108,9 @@
   </gazebo>
   <gazebo reference="r_hip_pitch_link">
-    <kp>100000.0</kp>
-    <kd>10.0</kd>
-    <mu1>0.1</mu1>
-    <maxVel>10.0</maxVel>
-    <minDepth>0.001</minDepth>
+    <kp>1000000.0</kp>
+    <kd>100.0</kd>
+    <mu1>0.1</mu1>
+    <maxVel>10.0</maxVel>
+    <minDepth>0.0001</minDepth>
     <maxContacts>6</maxContacts>
     <dampingFactor>0.0</dampingFactor>
@@ -119,9 +119,9 @@
   </gazebo>
   <gazebo reference="r_knee_link">
-    <kp>100000.0</kp>
-    <kd>10.0</kd>
-    <mu1>0.1</mu1>
-    <maxVel>10.0</maxVel>
-    <minDepth>0.001</minDepth>
+    <kp>1000000.0</kp>
+    <kd>100.0</kd>
+    <mu1>0.1</mu1>
+    <maxVel>10.0</maxVel>
+    <minDepth>0.0001</minDepth>
     <maxContacts>6</maxContacts>
     <dampingFactor>0.0</dampingFactor>
@@ -130,9 +130,9 @@
   </gazebo>
   <gazebo reference="r_ank_pitch_link">
-    <kp>100000.0</kp>
-    <kd>10.0</kd>
-    <mu1>0.1</mu1>
-    <maxVel>10.0</maxVel>
-    <minDepth>0.001</minDepth>
+    <kp>1000000.0</kp>
+    <kd>100.0</kd>
+    <mu1>0.1</mu1>
+    <maxVel>10.0</maxVel>
+    <minDepth>0.0001</minDepth>
     <maxContacts>6</maxContacts>
     <dampingFactor>0.0</dampingFactor>
@@ -141,9 +141,9 @@
   </gazebo>
   <gazebo reference="r_ank_roll_link">
-    <kp>100000.0</kp>
-    <kd>10.0</kd>
+    <kp>1000000.0</kp>
+    <kd>100.0</kd>
     <mu1>1.0</mu1>
     <maxVel>10.0</maxVel>
-    <minDepth>0.001</minDepth>
+    <minDepth>0.0001</minDepth>
     <maxContacts>6</maxContacts>
     <dampingFactor>0.0</dampingFactor>
@@ -152,9 +152,9 @@
   </gazebo>
   <gazebo reference="r_sho_pitch_link">
-    <kp>100000.0</kp>
-    <kd>10.0</kd>
-    <mu1>0.1</mu1>
-    <maxVel>10.0</maxVel>
-    <minDepth>0.001</minDepth>
+    <kp>1000000.0</kp>
+    <kd>100.0</kd>
+    <mu1>0.1</mu1>
+    <maxVel>10.0</maxVel>
+    <minDepth>0.0001</minDepth>
     <maxContacts>6</maxContacts>
     <dampingFactor>0.0</dampingFactor>
@@ -163,9 +163,9 @@
   </gazebo>
   <gazebo reference="r_sho_roll_link">
-    <kp>100000.0</kp>
-    <kd>10.0</kd>
-    <mu1>0.1</mu1>
-    <maxVel>10.0</maxVel>
-    <minDepth>0.001</minDepth>
+    <kp>1000000.0</kp>
+    <kd>100.0</kd>
+    <mu1>0.1</mu1>
+    <maxVel>10.0</maxVel>
+    <minDepth>0.0001</minDepth>
     <maxContacts>6</maxContacts>
     <dampingFactor>0.0</dampingFactor>
@@ -174,9 +174,9 @@
   </gazebo>
   <gazebo reference="r_el_link">
-    <kp>100000.0</kp>
-    <kd>10.0</kd>
-    <mu1>0.1</mu1>
-    <maxVel>10.0</maxVel>
-    <minDepth>0.001</minDepth>
+    <kp>1000000.0</kp>
+    <kd>100.0</kd>
+    <mu1>0.1</mu1>
+    <maxVel>10.0</maxVel>
+    <minDepth>0.0001</minDepth>
     <maxContacts>6</maxContacts>
     <dampingFactor>0.0</dampingFactor>
@@ -185,9 +185,9 @@
   </gazebo>
   <gazebo reference="l_sho_pitch_link">
-    <kp>100000.0</kp>
-    <kd>10.0</kd>
-    <mu1>0.1</mu1>
-    <maxVel>10.0</maxVel>
-    <minDepth>0.001</minDepth>
+    <kp>1000000.0</kp>
+    <kd>100.0</kd>
+    <mu1>0.1</mu1>
+    <maxVel>10.0</maxVel>
+    <minDepth>0.0001</minDepth>
     <maxContacts>6</maxContacts>
     <dampingFactor>0.0</dampingFactor>
@@ -196,9 +196,9 @@
   </gazebo>
   <gazebo reference="l_sho_roll_link">
-    <kp>100000.0</kp>
-    <kd>10.0</kd>
-    <mu1>0.1</mu1>
-    <maxVel>10.0</maxVel>
-    <minDepth>0.001</minDepth>
+    <kp>1000000.0</kp>
+    <kd>100.0</kd>
+    <mu1>0.1</mu1>
+    <maxVel>10.0</maxVel>
+    <minDepth>0.0001</minDepth>
     <maxContacts>6</maxContacts>
     <dampingFactor>0.0</dampingFactor>
@@ -207,9 +207,9 @@
   </gazebo>
   <gazebo reference="l_el_link">
-    <kp>100000.0</kp>
-    <kd>10.0</kd>
-    <mu1>0.1</mu1>
-    <maxVel>10.0</maxVel>
-    <minDepth>0.001</minDepth>
+    <kp>1000000.0</kp>
+    <kd>100.0</kd>
+    <mu1>0.1</mu1>
+    <maxVel>10.0</maxVel>
+    <minDepth>0.0001</minDepth>
     <maxContacts>6</maxContacts>
     <dampingFactor>0.0</dampingFactor>
@@ -218,9 +218,9 @@
   </gazebo>
   <gazebo reference="head_pan_link">
-    <kp>100000.0</kp>
-    <kd>10.0</kd>
-    <mu1>0.1</mu1>
-    <maxVel>10.0</maxVel>
-    <minDepth>0.001</minDepth>
+    <kp>1000000.0</kp>
+    <kd>100.0</kd>
+    <mu1>0.1</mu1>
+    <maxVel>10.0</maxVel>
+    <minDepth>0.0001</minDepth>
     <maxContacts>6</maxContacts>
     <dampingFactor>0.0</dampingFactor>
@@ -229,9 +229,9 @@
   </gazebo>
   <gazebo reference="head_tilt_link">
-    <kp>100000.0</kp>
-    <kd>10.0</kd>
-    <mu1>0.1</mu1>
-    <maxVel>10.0</maxVel>
-    <minDepth>0.001</minDepth>
+    <kp>1000000.0</kp>
+    <kd>100.0</kd>
+    <mu1>0.1</mu1>
+    <maxVel>10.0</maxVel>
+    <minDepth>0.0001</minDepth>
     <maxContacts>6</maxContacts>
     <dampingFactor>0.0</dampingFactor>

File: op3_description/urdf/robotis_op3.inertia.xacro (robot description, xacro)
@@ -5,8 +5,7 @@
     <origin xyz="-0.01501 0.00013 0.06582"/>
     <mass value="1.34928"/>
-    <inertia ixx="0.00340499" ixy="0.00000572" ixz="-0.00004256"
-      iyy="0.00296939" iyz="-0.00000059"
+    <inertia ixx="0.00340499" ixy="0.0" ixz="0.0"
+      iyy="0.00296939" iyz="0.0"
       izz="0.00317331"/>
-    <!--<inertia ixx="1.0" ixy="0.0" ixz="0.0" iyy="1.0" iyz="0.0" izz="1.0" />-->
   </xacro:macro>
   <!-- right hip yaw link -->
@@ -14,7 +13,7 @@
     <origin xyz="-0.00157 0.00000 -0.00774"/>
     <mass value="0.01181"/>
-    <inertia ixx="0.00000151" ixy="0.0" ixz="0.00000001"
-      iyy="0.00000430" iyz="0.0"
-      izz="0.00000412"/>
+    <inertia ixx="0.00001" ixy="0.0" ixz="0.0"
+      iyy="0.00001" iyz="0.0"
+      izz="0.00001"/>
   </xacro:macro>
   <!-- right hip roll link -->
@@ -22,6 +21,6 @@
     <origin xyz="0.00388 -0.00028 -0.01214"/>
     <mass value="0.17886"/>
-    <inertia ixx="0.00004661" ixy="0.00000101" ixz="-0.00000131"
-      iyy="0.00012523" iyz="0.00000006"
+    <inertia ixx="0.00004661" ixy="0.0" ixz="0.0"
+      iyy="0.00012523" iyz="0.0"
       izz="0.00010857"/>
   </xacro:macro>
@@ -30,6 +29,6 @@
     <origin xyz="0.00059 0.01901 -0.08408"/>
     <mass value="0.11543"/>
-    <inertia ixx="0.00010499" ixy="0.00000001" ixz="-0.00000071"
-      iyy="0.00009613" iyz="-0.00000353"
+    <inertia ixx="0.00010499" ixy="0.0" ixz="0.0"
+      iyy="0.00009613" iyz="0.0"
       izz="0.00002493"/>
   </xacro:macro>
@@ -46,6 +45,6 @@
     <origin xyz="-0.02022 0.01872 0.01214"/>
     <mass value="0.17886"/>
-    <inertia ixx="0.00004661" ixy="0.00000101" ixz="0.00000131"
-      iyy="0.00012523" iyz="-0.00000006"
+    <inertia ixx="0.00004661" ixy="0.0" ixz="0.0"
+      iyy="0.00012523" iyz="0.0"
       izz="0.00010857"/>
   </xacro:macro>
@@ -54,6 +53,6 @@
     <origin xyz="0.02373 -0.01037 -0.02760"/>
     <mass value="0.06934"/>
-    <inertia ixx="0.00004034" ixy="0.00000019" ixz="0.00000012"
-      iyy="0.00007874" iyz="-0.00000101"
+    <inertia ixx="0.00004034" ixy="0.0" ixz="0.0"
+      iyy="0.00007874" iyz="0.0"
       izz="0.00011579"/>
   </xacro:macro>
@@ -62,7 +61,7 @@
     <origin xyz="-0.00157 0.00000 -0.00774"/>
     <mass value="0.01181"/>
-    <inertia ixx="0.00000151" ixy="0.0" ixz="0.00000001"
-      iyy="0.00000430" iyz="0.0"
-      izz="0.00000412"/>
+    <inertia ixx="0.00001" ixy="0.0" ixz="0.0"
+      iyy="0.00001" iyz="0.0"
+      izz="0.00001"/>
   </xacro:macro>
   <!-- left hip roll link -->
@@ -70,6 +69,6 @@
     <origin xyz="0.00388 0.00028 -0.01214"/>
     <mass value="0.17886"/>
-    <inertia ixx="0.00004661" ixy="-0.00000101" ixz="-0.00000131"
-      iyy="0.00012523" iyz="-0.00000006"
+    <inertia ixx="0.00004661" ixy="0.0" ixz="0.0"
+      iyy="0.00012523" iyz="0.0"
       izz="0.00010857"/>
   </xacro:macro>
@@ -78,6 +77,6 @@
     <origin xyz="0.00059 -0.01901 -0.08408"/>
     <mass value="0.11543"/>
-    <inertia ixx="0.00010499" ixy="-0.00000001" ixz="-0.00000071"
-      iyy="0.00009613" iyz="0.00000353"
+    <inertia ixx="0.00010499" ixy="0.0" ixz="0.0"
+      iyy="0.00009613" iyz="0.0"
       izz="0.00002493"/>
   </xacro:macro>
@@ -94,6 +93,6 @@
     <origin xyz="-0.02022 -0.01872 0.01214"/>
     <mass value="0.17886"/>
-    <inertia ixx="0.00004661" ixy="-0.00000101" ixz="0.00000131"
-      iyy="0.00012523" iyz="0.00000006"
+    <inertia ixx="0.00004661" ixy="0.0" ixz="0.0"
+      iyy="0.00012523" iyz="0.0"
       izz="0.00010857"/>
   </xacro:macro>
@@ -102,6 +101,6 @@
     <origin xyz="0.02373 0.01037 -0.02760"/>
     <mass value="0.06934"/>
-    <inertia ixx="0.00004034" ixy="-0.00000019" ixz="0.00000012"
-      iyy="0.00007874" iyz="0.00000101"
+    <inertia ixx="0.00004034" ixy="0.0" ixz="0.0"
+      iyy="0.00007874" iyz="0.0"
       izz="0.00011579"/>
   </xacro:macro>
@@ -110,7 +109,7 @@
     <origin xyz="0.0 -0.00823 -0.00233"/>
     <mass value="0.01176"/>
-    <inertia ixx="0.00000165" ixy="0.0" ixz="0.0"
-      iyy="0.00000387" iyz="-0.00000031"
-      izz="0.00000397"/>
+    <inertia ixx="0.00001" ixy="0.0" ixz="0.0"
+      iyy="0.00001" iyz="0.0"
+      izz="0.00001"/>
   </xacro:macro>
   <!-- right shoulder roll joint -->
@@ -118,6 +117,6 @@
     <origin xyz="-0.01844 -0.04514 0.00028"/>
     <mass value="0.17758"/>
-    <inertia ixx="0.00022804" ixy="0.00000001" ixz="0.00000003"
-      iyy="0.00003042" iyz="-0.00000059"
+    <inertia ixx="0.00022804" ixy="0.0" ixz="0.0"
+      iyy="0.00003042" iyz="0.0"
       izz="0.00023474"/>
   </xacro:macro>
@@ -134,7 +133,7 @@
     <origin xyz="0.0 0.00823 -0.00233"/>
     <mass value="0.01176"/>
-    <inertia ixx="0.00000165" ixy="0.0" ixz="0.0"
-      iyy="0.00000387" iyz="0.00000031"
-      izz="0.00000397"/>
+    <inertia ixx="0.00001" ixy="0.0" ixz="0.0"
+      iyy="0.00001" iyz="0.0"
+      izz="0.00001"/>
   </xacro:macro>
   <!-- left shoulder roll joint -->
@@ -158,7 +157,7 @@
     <origin xyz="0.00233 0.00000 0.00823"/>
     <mass value="0.01176"/>
-    <inertia ixx="0.00000397" ixy="0.0" ixz="-0.00000031"
-      iyy="0.00000165" iyz="0.0"
-      izz="0.00000387"/>
+    <inertia ixx="0.00001" ixy="0.0" ixz="0.0"
+      iyy="0.00001" iyz="0.0"
+      izz="0.00001"/>
   </xacro:macro>
   <!-- head pitch joint -->

Commit message: Fix head

File: op3_description/urdf/robotis_op3.gazebo.xacro (robot description, xacro)
@@ -520,5 +520,5 @@
   </gazebo>
   <!-- head camera -->
-  <gazebo reference="cam_gazebo_link">
+  <gazebo reference="cam_link">
     <sensor name="camera" type="camera">
       <pose>0.050000 -0.010000 0.000000 0 0.000000 0</pose>
@@ -543,5 +543,5 @@
         <imageTopicName>image_raw</imageTopicName>
         <cameraInfoTopicName>camera_info</cameraInfoTopicName>
-        <frameName>cam_link</frameName>
+        <frameName>cam_optical_link</frameName>
         <hackBaseline>0.07</hackBaseline>
         <distortionK1>0.0</distortionK1>

File: op3_description/urdf/robotis_op3.inertia.xacro (robot description, xacro)
@@ -155,5 +155,5 @@
   <!-- head yaw joint -->
   <xacro:macro name="insert_inertia_head_pan_link">
-    <origin xyz="0.00233 0.00000 0.00823"/>
+    <origin xyz="0.0 0.0 0.0"/>
     <mass value="0.01176"/>
     <inertia ixx="0.00001" ixy="0.0" ixz="0.0"
@@ -163,5 +163,5 @@
   <!-- head pitch joint -->
   <xacro:macro name="insert_inertia_head_tilt_link">
-    <origin xyz="0.00230 -0.01863 0.02770"/>
+    <origin xyz="0.00230 0.0 0.0285"/>
     <mass value="0.13631"/>
     <inertia ixx="0.00010612" ixy="0.00000011" ixz="-0.00000910"

File: op3_description/urdf/robotis_op3.structure.head.xacro (robot description, xacro)
@@ -10,5 +10,5 @@
       <parent link="${parent}"/>
       <child link="head_pan_link"/>
-      <origin xyz="-0.001 0.0 0.1365" rpy="0 0 0"/>
+      <origin xyz="-0.001 0.0 0.165" rpy="0 0 0"/>
       <axis xyz="0 0 1"/>
       <limit effort="3.40" velocity="3.14" lower="${-pi*0.9}" upper="${pi*0.9}"/>
@@ -32,5 +32,5 @@
       <parent link="head_pan_link"/>
       <child link="head_tilt_link"/>
-      <origin xyz="0.010 0.019 0.0285" rpy="0 0 0"/>
+      <origin xyz="0.010 0.0 0.0" rpy="0 0 0"/>
       <axis xyz="0 -1 0"/>
       <limit effort="3.40" velocity="3.14" lower="${-pi*0.9}" upper="${pi*0.9}"/>
@@ -51,18 +51,18 @@
     </link>
     <!-- camera joint -->
+    <joint name="cam_optical" type="fixed">
+      <origin xyz="0.01425 0.0 0.04975" rpy="${-pi*0.5} 0 ${-pi*0.5}"/>
+      <parent link="head_tilt_link"/>
+      <child link="cam_optical_link"/>
+    </joint>
     <joint name="cam" type="fixed">
-      <origin xyz="0.01425 -0.019 0.04975" rpy="${-pi*0.5} 0 ${-pi*0.5}"/>
+      <origin xyz="0.01425 0.0 0.04975" rpy="0 0 0"/>
       <parent link="head_tilt_link"/>
       <child link="cam_link"/>
     </joint>
-    <joint name="cam_gazebo" type="fixed">
-      <origin xyz="0.01425 -0.019 0.04975" rpy="0 0 0"/>
-      <parent link="head_tilt_link"/>
-      <child link="cam_gazebo_link"/>
-    </joint>
+    <!-- camera link -->
+    <link name="cam_optical_link"/>
     <!-- camera link -->
     <link name="cam_link"/>
-    <!-- camera link -->
-    <link name="cam_gazebo_link"/>
   </xacro:macro>
 </robot>

File: op3_description/urdf/robotis_op3.visuals.xacro (robot description, xacro)
@@ -310,5 +310,5 @@
   <!-- head yaw joint -->
   <xacro:macro name="insert_mesh_head_pan_link">
-    <origin xyz="0 0 0" rpy="0 0 0"/>
+    <origin xyz="0 0 -0.0285" rpy="0 0 0"/>
     <geometry>
       <mesh filename="package://op3_description/meshes/h1.stl" scale="0.001 0.001 0.001"/>
@@ -319,5 +319,5 @@
   </xacro:macro>
   <xacro:macro name="insert_box_head_pan_link">
-    <origin xyz="0.0038 -0.0000 0.0155" rpy="0.0000 -0.0000 -0.0000"/>
+    <origin xyz="0.0038 -0.0000 -0.013" rpy="0.0000 -0.0000 -0.0000"/>
     <geometry>
       <box size="0.0325 0.0420 0.0310"/>
@@ -329,5 +329,5 @@
   <!-- head yaw joint -->
   <xacro:macro name="insert_mesh_head_tilt_link">
-    <origin xyz="0 0 0" rpy="0 0 0"/>
+    <origin xyz="0 0.019 0" rpy="0 0 0"/>
     <geometry>
       <mesh filename="package://op3_description/meshes/h2.stl" scale="0.001 0.001 0.001"/>
@@ -338,5 +338,5 @@
   </xacro:macro>
   <xacro:macro name="insert_box_head_tilt_link">
-    <origin xyz="0.0060 -0.0190 0.0278" rpy="0.0000 -0.0000 -0.0000"/>
+    <origin xyz="0.0060 0 0.0278" rpy="0.0000 -0.0000 -0.0000"/>
     <geometry>
       <box size="0.0445 0.0940 0.0780"/>
