Commit message: Fix left arm

File: op3_description/urdf/robotis_op3.inertia.xacro (robot description, xacro)
@@ -131,5 +131,5 @@
   <!-- left shoulder pitch joint -->
   <xacro:macro name="insert_inertia_l_sho_pitch_link">
-    <origin xyz="0.0 0.00823 -0.00233"/>
+    <origin xyz="0.0 0.0 0.0"/>
     <mass value="0.01176"/>
     <inertia ixx="0.00001" ixy="0.0" ixz="0.0"
@@ -139,5 +139,5 @@
   <!-- left shoulder roll joint -->
   <xacro:macro name="insert_inertia_l_sho_roll_link">
-    <origin xyz="-0.01844 0.04514 0.00028"/>
+    <origin xyz="0.0 0.04514 0.00028"/>
     <mass value="0.17758"/>
     <inertia ixx="0.00022804" ixy="-0.00000001" ixz="0.00000003"
@@ -147,5 +147,5 @@
   <!-- left elbow joint -->
   <xacro:macro name="insert_inertia_l_el_link">
-    <origin xyz="-0.01900 0.07033 0.00380"/>
+    <origin xyz="0.0 0.07033 0.00380"/>
     <mass value="0.04127"/>
     <inertia ixx="0.00006196" ixy="0.0" ixz="0.0"

File: op3_description/urdf/robotis_op3.structure.larm.xacro (robot description, xacro)
@@ -10,5 +10,5 @@
       <parent link="${parent}"/>
       <child link="l_sho_pitch_link"/>
-      <origin xyz="-0.001 0.06 0.111" rpy="0 0 0"/>
+      <origin xyz="-0.001 0.0885 0.111" rpy="0 0 0"/>
       <axis xyz="0 1 0"/>
       <limit effort="3.40" velocity="3.14" lower="${-pi*0.9}" upper="${pi*0.9}"/>
@@ -32,5 +32,5 @@
       <parent link="l_sho_pitch_link"/>
       <child link="l_sho_roll_link"/>
-      <origin xyz="0.019 0.0285 -0.010" rpy="0 0 0"/>
+      <origin xyz="0.0 0.0 -0.010" rpy="0 0 0"/>
       <axis xyz="-1 0 0"/>
       <limit effort="3.40" velocity="3.14" lower="${-pi*0.9}" upper="${pi*0.9}"/>

File: op3_description/urdf/robotis_op3.visuals.xacro (robot description, xacro)
@@ -262,5 +262,5 @@
   <!-- left shoulder pitch joint -->
   <xacro:macro name="insert_mesh_l_sho_pitch_link">
-    <origin xyz="0 0 0" rpy="0 0 0"/>
+    <origin xyz="0 -0.0285 0" rpy="0 0 0"/>
     <geometry>
       <mesh filename="package://op3_description/meshes/la1.stl" scale="0.001 0.001 0.001"/>
@@ -271,12 +271,12 @@
   </xacro:macro>
   <xacro:macro name="insert_box_l_sho_pitch_link">
-    <origin xyz="0.0000 0.0155 -0.0038" rpy="0.0000 -0.0000 -0.0000"/>
+    <origin xyz="0.0000 -0.013 -0.0038" rpy="0.0000 -0.0000 -0.0000"/>
     <geometry>
       <box size="0.0420 0.0310 0.0325"/>
     </geometry>
   </xacro:macro>
-  <!-- left shoulder pitch joint -->
+  <!-- left shoulder roll joint -->
   <xacro:macro name="insert_mesh_l_sho_roll_link">
-    <origin xyz="0 0 0" rpy="0 0 0"/>
+    <origin xyz="0.019 0 0" rpy="0 0 0"/>
     <geometry>
       <mesh filename="package://op3_description/meshes/la2.stl" scale="0.001 0.001 0.001"/>
@@ -287,5 +287,5 @@
   </xacro:macro>
   <xacro:macro name="insert_box_l_sho_roll_link">
-    <origin xyz="-0.0168 0.0452 0.0007" rpy="0.0000 -0.0000 -0.0000"/>
+    <origin xyz="0.0022 0.0452 0.0007" rpy="0.0000 -0.0000 -0.0000"/>
     <geometry>
       <box size="0.0424 0.1129 0.0301"/>
@@ -294,5 +294,5 @@
   <!-- left elbow joint -->
   <xacro:macro name="insert_mesh_l_el_link">
-    <origin xyz="0 0 0" rpy="0 0 0"/>
+    <origin xyz="0.019 0 0" rpy="0 0 0"/>
     <geometry>
       <mesh filename="package://op3_description/meshes/la3.stl" scale="0.001 0.001 0.001"/>
@@ -303,5 +303,5 @@
   </xacro:macro>
   <xacro:macro name="insert_box_l_el_link">
-    <origin xyz="-0.0190 0.0720 0.0000" rpy="0.0000 -0.0000 -0.0000"/>
+    <origin xyz="0.0 0.0720 0.0000" rpy="0.0000 -0.0000 -0.0000"/>
     <geometry>
       <box size="0.0420 0.1490 0.0300"/>

Commit message: Fix right arm

File: op3_description/urdf/robotis_op3.inertia.xacro (robot description, xacro)
@@ -107,5 +107,5 @@
   <!-- right shoulder pitch joint -->
   <xacro:macro name="insert_inertia_r_sho_pitch_link">
-    <origin xyz="0.0 -0.00823 -0.00233"/>
+    <origin xyz="0.0 0.0 0.0"/>
     <mass value="0.01176"/>
     <inertia ixx="0.00001" ixy="0.0" ixz="0.0"
@@ -115,5 +115,5 @@
   <!-- right shoulder roll joint -->
   <xacro:macro name="insert_inertia_r_sho_roll_link">
-    <origin xyz="-0.01844 -0.04514 0.00028"/>
+    <origin xyz="0.0 -0.04514 0.00028"/>
     <mass value="0.17758"/>
     <inertia ixx="0.00022804" ixy="0.0" ixz="0.0"
@@ -123,5 +123,5 @@
   <!-- right elbow joint -->
   <xacro:macro name="insert_inertia_r_el_link">
-    <origin xyz="-0.01900 -0.07033 0.00380"/>
+    <origin xyz="0.0 -0.07033 0.00380"/>
     <mass value="0.04127"/>
     <inertia ixx="0.00006196" ixy="0.0" ixz="0.0"

File: op3_description/urdf/robotis_op3.structure.rarm.xacro (robot description, xacro)
@@ -10,5 +10,5 @@
       <parent link="${parent}"/>
       <child link="r_sho_pitch_link"/>
-      <origin xyz="-0.001 -0.06 0.111" rpy="0 0 0"/>
+      <origin xyz="-0.001 -0.0885 0.111" rpy="0 0 0"/>
       <axis xyz="0 -1 0"/>
       <limit effort="3.40" velocity="3.14" lower="${-pi*0.9}" upper="${pi*0.9}"/>
@@ -32,5 +32,5 @@
       <parent link="r_sho_pitch_link"/>
       <child link="r_sho_roll_link"/>
-      <origin xyz="0.019 -0.0285 -0.010" rpy="0 0 0"/>
+      <origin xyz="0.0 0.0 -0.010" rpy="0 0 0"/>
       <axis xyz="-1 0 0"/>
       <limit effort="3.40" velocity="3.14" lower="${-pi*0.9}" upper="${pi*0.9}"/>

File: op3_description/urdf/robotis_op3.visuals.xacro (robot description, xacro)
@@ -214,5 +214,5 @@
   <!-- right shoulder pitch joint -->
   <xacro:macro name="insert_mesh_r_sho_pitch_link">
-    <origin xyz="0 0 0" rpy="0 0 0"/>
+    <origin xyz="0 0.0285 0" rpy="0 0 0"/>
     <geometry>
       <mesh filename="package://op3_description/meshes/ra1.stl" scale="0.001 0.001 0.001"/>
@@ -223,12 +223,12 @@
   </xacro:macro>
   <xacro:macro name="insert_box_r_sho_pitch_link">
-    <origin xyz="-0.0000 -0.0155 -0.0038" rpy="0.0000 -0.0000 -0.0000"/>
+    <origin xyz="-0.0000 0.013 -0.0038" rpy="0.0000 -0.0000 -0.0000"/>
     <geometry>
       <box size="0.0420 0.0310 0.0325"/>
     </geometry>
   </xacro:macro>
-  <!-- right shoulder pitch joint -->
+  <!-- right shoulder roll joint -->
   <xacro:macro name="insert_mesh_r_sho_roll_link">
-    <origin xyz="0 0 0" rpy="0 0 0"/>
+    <origin xyz="0.019 0 0" rpy="0 0 0"/>
     <geometry>
       <mesh filename="package://op3_description/meshes/ra2.stl" scale="0.001 0.001 0.001"/>
@@ -239,5 +239,5 @@
   </xacro:macro>
   <xacro:macro name="insert_box_r_sho_roll_link">
-    <origin xyz="-0.0168 -0.0452 0.0007" rpy="0.0000 -0.0000 -0.0000"/>
+    <origin xyz="0.0022 -0.0452 0.0007" rpy="0.0000 -0.0000 -0.0000"/>
     <geometry>
       <box size="0.0424 0.1129 0.0301"/>
@@ -246,5 +246,5 @@
   <!-- right elbow joint -->
   <xacro:macro name="insert_mesh_r_el_link">
-    <origin xyz="0 0 0" rpy="0 0 0"/>
+    <origin xyz="0.019 0 0" rpy="0 0 0"/>
     <geometry>
       <mesh filename="package://op3_description/meshes/ra3.stl" scale="0.001 0.001 0.001"/>
@@ -255,5 +255,5 @@
   </xacro:macro>
   <xacro:macro name="insert_box_r_el_link">
-    <origin xyz="-0.0190 -0.0720 0.0000" rpy="0.0000 -0.0000 -0.0000"/>
+    <origin xyz="0.0 -0.0720 0.0000" rpy="0.0000 -0.0000 -0.0000"/>
     <geometry>
       <box size="0.0420 0.1490 0.0300"/>

Commit message: Fix left leg

File: op3_description/urdf/robotis_op3.inertia.xacro (robot description, xacro)
@@ -59,5 +59,5 @@
   <!-- left hip yaw link -->
   <xacro:macro name="insert_inertia_l_hip_yaw_link">
-    <origin xyz="-0.00157 0.00000 -0.00774"/>
+    <origin xyz="-0.00157 0.00000 0.02076"/>
     <mass value="0.01181"/>
     <inertia ixx="0.00001" ixy="0.0" ixz="0.0"
@@ -67,5 +67,5 @@
   <!-- left hip roll link -->
   <xacro:macro name="insert_inertia_l_hip_roll_link">
-    <origin xyz="0.00388 0.00028 -0.01214"/>
+    <origin xyz="-0.0201 0.00028 -0.01214"/>
     <mass value="0.17886"/>
     <inertia ixx="0.00004661" ixy="0.0" ixz="0.0"
@@ -75,5 +75,5 @@
   <!-- left hip pitch link -->
   <xacro:macro name="insert_inertia_l_hip_pitch_link">
-    <origin xyz="0.00059 -0.01901 -0.08408"/>
+    <origin xyz="0.00059 -0.00001 -0.08408"/>
     <mass value="0.11543"/>
     <inertia ixx="0.00010499" ixy="0.0" ixz="0.0"
@@ -83,5 +83,5 @@
   <!-- left knee link -->
   <xacro:macro name="insert_inertia_l_knee_link">
-    <origin xyz="0.00000 -0.02151 -0.05500"/>
+    <origin xyz="0.00000 -0.00251 -0.05500"/>
     <mass value="0.04015"/>
     <inertia ixx="0.00003715" ixy="0.0" ixz="0.0"
@@ -91,5 +91,5 @@
   <!-- left ankle pitch link -->
   <xacro:macro name="insert_inertia_l_ank_pitch_link">
-    <origin xyz="-0.02022 -0.01872 0.01214"/>
+    <origin xyz="-0.02022 0.00028 0.01214"/>
     <mass value="0.17886"/>
     <inertia ixx="0.00004661" ixy="0.0" ixz="0.0"
@@ -99,5 +99,5 @@
   <!-- left ankle roll link -->
   <xacro:macro name="insert_inertia_l_ank_roll_link">
-    <origin xyz="0.02373 0.01037 -0.02760"/>
+    <origin xyz="-0.00037 0.01037 -0.02760"/>
     <mass value="0.06934"/>
     <inertia ixx="0.00004034" ixy="0.0" ixz="0.0"

File: op3_description/urdf/robotis_op3.structure.lleg.xacro (robot description, xacro)
@@ -10,5 +10,5 @@
       <parent link="${parent}"/>
       <child link="l_hip_yaw_link"/>
-      <origin xyz="0.0 0.035 0.0" rpy="0 0 0"/>
+      <origin xyz="0.0 0.035 -0.0285" rpy="0 0 0"/>
       <axis xyz="0 0 -1"/>
       <limit effort="3.40" velocity="3.14" lower="${-pi*0.9}" upper="${pi*0.9}"/>
@@ -32,5 +32,5 @@
       <parent link="l_hip_yaw_link"/>
       <child link="l_hip_roll_link"/>
-      <origin xyz="-0.024 0.0 -0.0285" rpy="0 0 0"/>
+      <origin xyz="0.0 0.0 0.0" rpy="0 0 0"/>
       <axis xyz="-1 0 0"/>
       <limit effort="3.40" velocity="3.14" lower="${-pi*0.9}" upper="${pi*0.9}"/>
@@ -54,5 +54,5 @@
       <parent link="l_hip_roll_link"/>
       <child link="l_hip_pitch_link"/>
-      <origin xyz="0.0241 0.019 0.0" rpy="0 0 0"/>
+      <origin xyz="0.0001 0.0 0.0" rpy="0 0 0"/>
       <axis xyz="0 1 0"/>
       <limit effort="3.40" velocity="3.14" lower="${-pi*0.9}" upper="${pi*0.9}"/>
@@ -120,5 +120,5 @@
       <parent link="l_ank_pitch_link"/>
       <child link="l_ank_roll_link"/>
-      <origin xyz="-0.0241 -0.019 0" rpy="0 0 0"/>
+      <origin xyz="0 0 0" rpy="0 0 0"/>
       <axis xyz="1 0 0"/>
       <limit effort="3.40" velocity="3.14" lower="${-pi*0.9}" upper="${pi*0.9}"/>

File: op3_description/urdf/robotis_op3.visuals.xacro (robot description, xacro)
@@ -118,5 +118,5 @@
   <!-- left hip yaw link -->
   <xacro:macro name="insert_mesh_l_hip_yaw_link">
-    <origin xyz="0 0 0" rpy="0 0 0"/>
+    <origin xyz="0 0 0.0285" rpy="0 0 0"/>
     <geometry>
       <mesh filename="package://op3_description/meshes/ll1.stl" scale="0.001 0.001 0.001"/>
@@ -127,5 +127,5 @@
   </xacro:macro>
   <xacro:macro name="insert_box_l_hip_yaw_link">
-    <origin xyz="-0.0015 0.0000 -0.0155" rpy="0.0000 -0.0000 -0.0000"/>
+    <origin xyz="-0.0015 0.0000 0.013" rpy="0.0000 -0.0000 -0.0000"/>
     <geometry>
       <box size="0.0450 0.0250 0.0310"/>
@@ -134,5 +134,5 @@
   <!-- left hip roll link -->
   <xacro:macro name="insert_mesh_l_hip_roll_link">
-    <origin xyz="0 0 0" rpy="0 0 0"/>
+    <origin xyz="-0.024 0 0" rpy="0 0 0"/>
     <geometry>
       <mesh filename="package://op3_description/meshes/ll2.stl" scale="0.001 0.001 0.001"/>
@@ -143,5 +143,5 @@
   </xacro:macro>
   <xacro:macro name="insert_box_l_hip_roll_link">
-    <origin xyz="0.0039 0.0022 -0.0120" rpy="0.0000 -0.0000 -0.0000"/>
+    <origin xyz="-0.0201 0.0022 -0.0120" rpy="0.0000 -0.0000 -0.0000"/>
     <geometry>
       <box size="0.0798 0.0424 0.0465"/>
@@ -150,5 +150,5 @@
   <!-- left hip pitch link -->
   <xacro:macro name="insert_mesh_l_hip_pitch_link">
-    <origin xyz="0 0 0" rpy="0 0 0"/>
+    <origin xyz="0.0 0.019 0" rpy="0 0 0"/>
     <geometry>
       <mesh filename="package://op3_description/meshes/ll3.stl" scale="0.001 0.001 0.001"/>
@@ -159,5 +159,5 @@
   </xacro:macro>
   <xacro:macro name="insert_box_l_hip_pitch_link">
-    <origin xyz="0.0004 -0.0188 -0.0595" rpy="0.0000 -0.0000 -0.0000"/>
+    <origin xyz="0.0004 0.0002 -0.0595" rpy="0.0000 -0.0000 -0.0000"/>
     <geometry>
       <box size="0.0309 0.0464 0.1239"/>
@@ -166,5 +166,5 @@
   <!-- left knee link -->
   <xacro:macro name="insert_mesh_l_knee_link">
-    <origin xyz="0 0 0" rpy="0 0 0"/>
+    <origin xyz="0 0.019 0" rpy="0 0 0"/>
     <geometry>
       <mesh filename="package://op3_description/meshes/ll4.stl" scale="0.001 0.001 0.001"/>
@@ -175,5 +175,5 @@
   </xacro:macro>
   <xacro:macro name="insert_box_l_knee_link">
-    <origin xyz="-0.0000 -0.0200 -0.0550" rpy="0.0000 -0.0000 -0.0000"/>
+    <origin xyz="0.0 -0.001 -0.0550" rpy="0.0000 -0.0000 -0.0000"/>
     <geometry>
       <box size="0.0300 0.0440 0.1150"/>
@@ -182,5 +182,5 @@
   <!-- left ankle pitch link -->
   <xacro:macro name="insert_mesh_l_ank_pitch_link">
-    <origin xyz="0 0 0" rpy="0 0 0"/>
+    <origin xyz="0 0.019 0" rpy="0 0 0"/>
     <geometry>
       <mesh filename="package://op3_description/meshes/ll5.stl" scale="0.001 0.001 0.001"/>
@@ -191,5 +191,5 @@
   </xacro:macro>
   <xacro:macro name="insert_box_l_ank_pitch_link">
-    <origin xyz="-0.0206 -0.0168 0.0120" rpy="0.0000 -0.0000 -0.0000"/>
+    <origin xyz="-0.0206 0.0022 0.0120" rpy="0.0000 -0.0000 -0.0000"/>
     <geometry>
       <box size="0.0790 0.0424 0.0465"/>
@@ -198,5 +198,5 @@
   <!-- left ankle roll link -->
   <xacro:macro name="insert_mesh_l_ank_roll_link">
-    <origin xyz="0 0 0" rpy="0 0 0"/>
+    <origin xyz="-0.0241 0 0" rpy="0 0 0"/>
     <geometry>
       <mesh filename="package://op3_description/meshes/ll6.stl" scale="0.001 0.001 0.001"/>
@@ -207,5 +207,5 @@
   </xacro:macro>
   <xacro:macro name="insert_box_l_ank_roll_link">
-    <origin xyz="0.0240 0.0125 -0.0140" rpy="0.0000 -0.0000 -0.0000"/>
+    <origin xyz="-0.0001 0.0125 -0.0140" rpy="0.0000 -0.0000 -0.0000"/>
     <geometry>
       <box size="0.1270 0.0800 0.0330"/>

Commit message: Fix right leg

File: op3_description/urdf/robotis_op3.inertia.xacro (robot description, xacro)
@@ -11,5 +11,5 @@
   <!-- right hip yaw link -->
   <xacro:macro name="insert_inertia_r_hip_yaw_link">
-    <origin xyz="-0.00157 0.00000 -0.00774"/>
+    <origin xyz="-0.00157 0.00000 0.02076"/>
     <mass value="0.01181"/>
     <inertia ixx="0.00001" ixy="0.0" ixz="0.0"
@@ -19,5 +19,5 @@
   <!-- right hip roll link -->
   <xacro:macro name="insert_inertia_r_hip_roll_link">
-    <origin xyz="0.00388 -0.00028 -0.01214"/>
+    <origin xyz="-0.0201 -0.00028 -0.01214"/>
     <mass value="0.17886"/>
     <inertia ixx="0.00004661" ixy="0.0" ixz="0.0"
@@ -27,5 +27,5 @@
   <!-- right hip pitch link -->
   <xacro:macro name="insert_inertia_r_hip_pitch_link">
-    <origin xyz="0.00059 0.01901 -0.08408"/>
+    <origin xyz="0.00059 0.00001 -0.08408"/>
     <mass value="0.11543"/>
     <inertia ixx="0.00010499" ixy="0.0" ixz="0.0"
@@ -35,5 +35,5 @@
   <!-- right knee link -->
   <xacro:macro name="insert_inertia_r_knee_link">
-    <origin xyz="0.00000 0.02151 -0.05500"/>
+    <origin xyz="0.00000 0.00251 -0.05500"/>
     <mass value="0.04015"/>
     <inertia ixx="0.00003715" ixy="0.0" ixz="0.0"
@@ -43,5 +43,5 @@
   <!-- right ankle pitch link -->
   <xacro:macro name="insert_inertia_r_ank_pitch_link">
-    <origin xyz="-0.02022 0.01872 0.01214"/>
+    <origin xyz="-0.02022 -0.00028 0.01214"/>
     <mass value="0.17886"/>
     <inertia ixx="0.00004661" ixy="0.0" ixz="0.0"
@@ -51,5 +51,5 @@
   <!-- right ankle roll link -->
   <xacro:macro name="insert_inertia_r_ank_roll_link">
-    <origin xyz="0.02373 -0.01037 -0.02760"/>
+    <origin xyz="-0.00037 -0.01037 -0.02760"/>
     <mass value="0.06934"/>
     <inertia ixx="0.00004034" ixy="0.0" ixz="0.0"

File: op3_description/urdf/robotis_op3.structure.rleg.xacro (robot description, xacro)
@@ -10,5 +10,5 @@
       <parent link="${parent}"/>
       <child link="r_hip_yaw_link"/>
-      <origin xyz="0.0 -0.035 0.0" rpy="0 0 0"/>
+      <origin xyz="0.0 -0.035 -0.0285" rpy="0 0 0"/>
       <axis xyz="0 0 -1"/>
       <limit effort="3.40" velocity="3.14" lower="${-pi*0.9}" upper="${pi*0.9}"/>
@@ -32,5 +32,5 @@
       <parent link="r_hip_yaw_link"/>
       <child link="r_hip_roll_link"/>
-      <origin xyz="-0.024 0.0 -0.0285" rpy="0 0 0"/>
+      <origin xyz="0.0 0.0 0.0" rpy="0 0 0"/>
       <axis xyz="-1 0 0"/>
       <limit effort="3.40" velocity="3.14" lower="${-pi*0.9}" upper="${pi*0.9}"/>
@@ -54,5 +54,5 @@
       <parent link="r_hip_roll_link"/>
       <child link="r_hip_pitch_link"/>
-      <origin xyz="0.0241 -0.019 0.0" rpy="0 0 0"/>
+      <origin xyz="0.0001 0.0 0.0" rpy="0 0 0"/>
       <axis xyz="0 -1 0"/>
       <limit effort="3.40" velocity="3.14" lower="${-pi*0.9}" upper="${pi*0.9}"/>
@@ -120,5 +120,5 @@
       <parent link="r_ank_pitch_link"/>
       <child link="r_ank_roll_link"/>
-      <origin xyz="-0.0241 0.019 0" rpy="0 0 0"/>
+      <origin xyz="0 0 0" rpy="0 0 0"/>
       <axis xyz="1 0 0"/>
       <limit effort="3.40" velocity="3.14" lower="${-pi*0.9}" upper="${pi*0.9}"/>

File: op3_description/urdf/robotis_op3.visuals.xacro (robot description, xacro)
@@ -22,5 +22,5 @@
   <!-- right hip yaw link -->
   <xacro:macro name="insert_mesh_r_hip_yaw_link">
-    <origin xyz="0 0 0" rpy="0 0 0"/>
+    <origin xyz="0 0 0.0285" rpy="0 0 0"/>
     <geometry>
       <mesh filename="package://op3_description/meshes/rl1.stl" scale="0.001 0.001 0.001"/>
@@ -31,5 +31,5 @@
   </xacro:macro>
   <xacro:macro name="insert_box_r_hip_yaw_link">
-    <origin xyz="-0.0015 0.0000 -0.0155" rpy="0.0000 -0.0000 -0.0000"/>
+    <origin xyz="-0.0015 0.0000 0.013" rpy="0.0000 -0.0000 -0.0000"/>
     <geometry>
       <box size="0.0450 0.0250 0.0310"/>
@@ -38,5 +38,5 @@
   <!-- right hip roll link -->
   <xacro:macro name="insert_mesh_r_hip_roll_link">
-    <origin xyz="0 0 0" rpy="0 0 0"/>
+    <origin xyz="-0.024 0 0" rpy="0 0 0"/>
     <geometry>
       <mesh filename="package://op3_description/meshes/rl2.stl" scale="0.001 0.001 0.001"/>
@@ -47,5 +47,5 @@
   </xacro:macro>
   <xacro:macro name="insert_box_r_hip_roll_link">
-    <origin xyz="0.0039 -0.0022 -0.0120" rpy="0.0000 -0.0000 -0.0000"/>
+    <origin xyz="-0.0201 -0.0022 -0.0120" rpy="0.0000 -0.0000 -0.0000"/>
     <geometry>
       <box size="0.0798 0.0424 0.0465"/>
@@ -54,5 +54,5 @@
   <!-- right hip pitch link -->
   <xacro:macro name="insert_mesh_r_hip_pitch_link">
-    <origin xyz="0 0 0" rpy="0 0 0"/>
+    <origin xyz="0 -0.019 0" rpy="0 0 0"/>
     <geometry>
       <mesh filename="package://op3_description/meshes/rl3.stl" scale="0.001 0.001 0.001"/>
@@ -63,5 +63,5 @@
   </xacro:macro>
   <xacro:macro name="insert_box_r_hip_pitch_link">
-    <origin xyz="0.0004 0.0188 -0.0595" rpy="0.0000 -0.0000 -0.0000"/>
+    <origin xyz="0.0004 -0.0002 -0.0595" rpy="0.0000 -0.0000 -0.0000"/>
     <geometry>
       <box size="0.0309 0.0464 0.1239"/>
@@ -70,5 +70,5 @@
   <!-- right knee link -->
   <xacro:macro name="insert_mesh_r_knee_link">
-    <origin xyz="0 0 0" rpy="0 0 0"/>
+    <origin xyz="0 -0.019 0" rpy="0 0 0"/>
     <geometry>
       <mesh filename="package://op3_description/meshes/rl4.stl" scale="0.001 0.001 0.001"/>
@@ -79,5 +79,5 @@
   </xacro:macro>
   <xacro:macro name="insert_box_r_knee_link">
-    <origin xyz="0.0000 0.0200 -0.0550" rpy="0.0000 -0.0000 -0.0000"/>
+    <origin xyz="0.0000 0.001 -0.0550" rpy="0.0000 -0.0000 -0.0000"/>
     <geometry>
       <box size="0.0300 0.0440 0.1150"/>
@@ -86,5 +86,5 @@
   <!-- right ankle pitch link -->
   <xacro:macro name="insert_mesh_r_ank_pitch_link">
-    <origin xyz="0 0 0" rpy="0 0 0"/>
+    <origin xyz="0 -0.019 0" rpy="0 0 0"/>
     <geometry>
       <mesh filename="package://op3_description/meshes/rl5.stl" scale="0.001 0.001 0.001"/>
@@ -95,5 +95,5 @@
   </xacro:macro>
   <xacro:macro name="insert_box_r_ank_pitch_link">
-    <origin xyz="-0.0202 0.0168 0.0120" rpy="0.0000 -0.0000 -0.0000"/>
+    <origin xyz="-0.0202 -0.0022 0.0120" rpy="0.0000 -0.0000 -0.0000"/>
     <geometry>
       <box size="0.0798 0.0424 0.0465"/>
@@ -102,5 +102,5 @@
   <!-- right ankle roll link -->
   <xacro:macro name="insert_mesh_r_ank_roll_link">
-    <origin xyz="0 0 0" rpy="0 0 0"/>
+    <origin xyz="-0.0241 0 0" rpy="0 0 0"/>
     <geometry>
       <mesh filename="package://op3_description/meshes/rl6.stl" scale="0.001 0.001 0.001"/>
@@ -111,5 +111,5 @@
   </xacro:macro>
   <xacro:macro name="insert_box_r_ank_roll_link">
-    <origin xyz="0.0240 -0.0125 -0.0140" rpy="0.0000 -0.0000 -0.0000"/>
+    <origin xyz="-0.0001 -0.0125 -0.0140" rpy="0.0000 -0.0000 -0.0000"/>
     <geometry>
       <box size="0.1270 0.0800 0.0330"/>
