Commit message: Parameter tuning

File: op3_description/urdf/robotis_op3.inertia.xacro (robot description, xacro)
@@ -126,5 +126,5 @@
     <mass value="0.04127"/>
     <inertia ixx="0.00006196" ixy="0.0" ixz="0.0"
-      iyy="0.00001231" iyz="0.00000372"
+      iyy="0.00001231" iyz="0.0"
       izz="0.00006854"/>
   </xacro:macro>
@@ -141,6 +141,6 @@
     <origin xyz="0.0 0.04514 0.00028"/>
     <mass value="0.17758"/>
-    <inertia ixx="0.00022804" ixy="-0.00000001" ixz="0.00000003"
-      iyy="0.00003042" iyz="0.00000059"
+    <inertia ixx="0.00022804" ixy="0.0" ixz="0.0"
+      iyy="0.00003042" iyz="0.0"
       izz="0.00023474"/>
   </xacro:macro>
@@ -150,5 +150,5 @@
     <mass value="0.04127"/>
     <inertia ixx="0.00006196" ixy="0.0" ixz="0.0"
-      iyy="0.00001231" iyz="-0.00000372"
+      iyy="0.00001231" iyz="0.0"
       izz="0.00006854"/>
   </xacro:macro>
@@ -165,6 +165,6 @@
     <origin xyz="0.00230 0.0 0.0285"/>
     <mass value="0.13631"/>
-    <inertia ixx="0.00010612" ixy="0.00000011" ixz="-0.00000910"
-      iyy="0.00008721" iyz="0.00000084"
+    <inertia ixx="0.00010612" ixy="0.0" ixz="0.0"
+      iyy="0.00008721" iyz="0.0"
       izz="0.00004529"/>
   </xacro:macro>

File: op3_description/urdf/robotis_op3.structure.head.xacro (robot description, xacro)
@@ -13,5 +13,5 @@
       <axis xyz="0 0 1"/>
       <limit effort="3.40" velocity="3.14" lower="${-pi*0.9}" upper="${pi*0.9}"/>
-      <dynamics damping="1.08" friction="0.0"/>
+      <dynamics damping="0.1" friction="0.1"/>
     </joint>
     <xacro:insert_transmission name="head_pan"/>
@@ -35,5 +35,5 @@
       <axis xyz="0 -1 0"/>
       <limit effort="3.40" velocity="3.14" lower="${-pi*0.9}" upper="${pi*0.9}"/>
-      <dynamics damping="1.08" friction="0.0"/>
+      <dynamics damping="0.1" friction="0.1"/>
     </joint>
     <xacro:insert_transmission name="head_tilt"/>

File: op3_description/urdf/robotis_op3.structure.larm.xacro (robot description, xacro)
@@ -13,5 +13,5 @@
       <axis xyz="0 1 0"/>
       <limit effort="3.40" velocity="3.14" lower="${-pi*0.9}" upper="${pi*0.9}"/>
-      <dynamics damping="1.08" friction="0.0"/>
+      <dynamics damping="0.1" friction="0.1"/>
     </joint>
     <xacro:insert_transmission name="l_sho_pitch"/>
@@ -35,5 +35,5 @@
       <axis xyz="-1 0 0"/>
       <limit effort="3.40" velocity="3.14" lower="${-pi*0.9}" upper="${pi*0.9}"/>
-      <dynamics damping="1.08" friction="0.0"/>
+      <dynamics damping="0.1" friction="0.1"/>
     </joint>
     <xacro:insert_transmission name="l_sho_roll"/>
@@ -57,5 +57,5 @@
       <axis xyz="1 0 0"/>
       <limit effort="3.40" velocity="3.14" lower="${-pi*0.9}" upper="${pi*0.9}"/>
-      <dynamics damping="1.08" friction="0.0"/>
+      <dynamics damping="0.1" friction="0.1"/>
     </joint>
     <xacro:insert_transmission name="l_el"/>

File: op3_description/urdf/robotis_op3.structure.lleg.xacro (robot description, xacro)
@@ -13,5 +13,5 @@
       <axis xyz="0 0 -1"/>
       <limit effort="3.40" velocity="3.14" lower="${-pi*0.9}" upper="${pi*0.9}"/>
-      <dynamics damping="1.08" friction="0.0"/>
+      <dynamics damping="0.1" friction="0.1"/>
     </joint>
     <xacro:insert_transmission name="l_hip_yaw"/>
@@ -35,5 +35,5 @@
       <axis xyz="-1 0 0"/>
       <limit effort="3.40" velocity="3.14" lower="${-pi*0.9}" upper="${pi*0.9}"/>
-      <dynamics damping="1.08" friction="0.0"/>
+      <dynamics damping="0.1" friction="0.1"/>
     </joint>
     <xacro:insert_transmission name="l_hip_roll"/>
@@ -57,5 +57,5 @@
       <axis xyz="0 1 0"/>
       <limit effort="3.40" velocity="3.14" lower="${-pi*0.9}" upper="${pi*0.9}"/>
-      <dynamics damping="1.08" friction="0.0"/>
+      <dynamics damping="0.1" friction="0.1"/>
     </joint>
     <xacro:insert_transmission name="l_hip_pitch"/>
@@ -79,5 +79,5 @@
       <axis xyz="0 1 0"/>
       <limit effort="3.40" velocity="3.14" lower="${-pi*0.9}" upper="${pi*0.9}"/>
-      <dynamics damping="1.08" friction="0.0"/>
+      <dynamics damping="0.1" friction="0.1"/>
     </joint>
     <xacro:insert_transmission name="l_knee"/>
@@ -101,5 +101,5 @@
       <axis xyz="0 -1 0"/>
       <limit effort="3.40" velocity="3.14" lower="${-pi*0.9}" upper="${pi*0.9}"/>
-      <dynamics damping="1.08" friction="0.0"/>
+      <dynamics damping="0.1" friction="0.1"/>
     </joint>
     <xacro:insert_transmission name="l_ank_pitch"/>
@@ -123,5 +123,5 @@
       <axis xyz="1 0 0"/>
       <limit effort="3.40" velocity="3.14" lower="${-pi*0.9}" upper="${pi*0.9}"/>
-      <dynamics damping="1.08" friction="0.0"/>
+      <dynamics damping="0.1" friction="0.1"/>
     </joint>
     <xacro:insert_transmission name="l_ank_roll"/>

File: op3_description/urdf/robotis_op3.structure.rarm.xacro (robot description, xacro)
@@ -13,5 +13,5 @@
       <axis xyz="0 -1 0"/>
       <limit effort="3.40" velocity="3.14" lower="${-pi*0.9}" upper="${pi*0.9}"/>
-      <dynamics damping="1.08" friction="0.0"/>
+      <dynamics damping="0.1" friction="0.1"/>
     </joint>
     <xacro:insert_transmission name="r_sho_pitch"/>
@@ -35,5 +35,5 @@
       <axis xyz="-1 0 0"/>
       <limit effort="3.40" velocity="3.14" lower="${-pi*0.9}" upper="${pi*0.9}"/>
-      <dynamics damping="1.08" friction="0.0"/>
+      <dynamics damping="0.1" friction="0.1"/>
     </joint>
     <xacro:insert_transmission name="r_sho_roll"/>
@@ -57,5 +57,5 @@
       <axis xyz="1 0 0"/>
       <limit effort="3.40" velocity="3.14" lower="${-pi*0.9}" upper="${pi*0.9}"/>
-      <dynamics damping="1.08" friction="0.0"/>
+      <dynamics damping="0.1" friction="0.1"/>
     </joint>
     <xacro:insert_transmission name="r_el"/>

File: op3_description/urdf/robotis_op3.structure.rleg.xacro (robot description, xacro)
@@ -13,5 +13,5 @@
       <axis xyz="0 0 -1"/>
       <limit effort="3.40" velocity="3.14" lower="${-pi*0.9}" upper="${pi*0.9}"/>
-      <dynamics damping="1.08" friction="0.0"/>
+      <dynamics damping="0.1" friction="0.1"/>
     </joint>
     <xacro:insert_transmission name="r_hip_yaw"/>
@@ -35,5 +35,5 @@
       <axis xyz="-1 0 0"/>
       <limit effort="3.40" velocity="3.14" lower="${-pi*0.9}" upper="${pi*0.9}"/>
-      <dynamics damping="1.08" friction="0.0"/>
+      <dynamics damping="0.1" friction="0.1"/>
     </joint>
     <xacro:insert_transmission name="r_hip_roll"/>
@@ -57,5 +57,5 @@
       <axis xyz="0 -1 0"/>
       <limit effort="3.40" velocity="3.14" lower="${-pi*0.9}" upper="${pi*0.9}"/>
-      <dynamics damping="1.08" friction="0.0"/>
+      <dynamics damping="0.1" friction="0.1"/>
     </joint>
     <xacro:insert_transmission name="r_hip_pitch"/>
@@ -79,5 +79,5 @@
       <axis xyz="0 -1 0"/>
       <limit effort="3.40" velocity="3.14" lower="${-pi*0.9}" upper="${pi*0.9}"/>
-      <dynamics damping="1.08" friction="0.0"/>
+      <dynamics damping="0.1" friction="0.1"/>
     </joint>
     <xacro:insert_transmission name="r_knee"/>
@@ -101,5 +101,5 @@
       <axis xyz="0 1 0"/>
       <limit effort="3.40" velocity="3.14" lower="${-pi*0.9}" upper="${pi*0.9}"/>
-      <dynamics damping="1.08" friction="0.0"/>
+      <dynamics damping="0.1" friction="0.1"/>
     </joint>
     <xacro:insert_transmission name="r_ank_pitch"/>
@@ -123,5 +123,5 @@
       <axis xyz="1 0 0"/>
       <limit effort="3.40" velocity="3.14" lower="${-pi*0.9}" upper="${pi*0.9}"/>
-      <dynamics damping="1.08" friction="0.0"/>
+      <dynamics damping="0.1" friction="0.1"/>
     </joint>
     <xacro:insert_transmission name="r_ank_roll"/>
